File: rsp02_module_CS_5_0V.sch (KiCad schematic (older format))
At the start: 5 parts, among them IC13 INA199A1DCKT_v2

Commit message: Update PCB
Parts:
- C25: footprint (none) -> Capacitor_SMD:C_0603_1608Metric
- IC13: footprint SOT65P210X110-6N -> Package_TO_SOT_SMD:SOT-363_SC-70-6
- R112, R113: footprint (none) -> Resistor_SMD:R_0603_1608Metric
- R114: footprint (none) -> Resistor_SMD:R_2512_6332Metric
Changed lines of the file:
@@
 F 0 "R114" V 5490 2500 50  0000 C CNN
 F 1 "0.04" V 5660 2500 50  0000 C CNN
-F 2 "" V 5500 2500 50  0001 C CNN
+F 2 "Resistor_SMD:R_2512_6332Metric" V 5500 2500 50  0001 C CNN
 F 3 "~" H 5570 2500 50  0001 C CNN
 	1    5570 2500
@@
 F 0 "R112" V 4830 4450 50  0000 C CNN
 F 1 "0" V 4750 4340 50  0000 C CNN
-F 2 "" V 4680 4340 50  0001 C CNN
+F 2 "Resistor_SMD:R_0603_1608Metric" V 4680 4340 50  0001 C CNN
 F 3 "~" H 4750 4340 50  0001 C CNN
 	1    4750 4340
@@
 F 0 "R113" V 4840 4640 50  0000 C CNN
 F 1 "0" V 4750 4540 50  0000 C CNN
-F 2 "" V 4680 4540 50  0001 C CNN
+F 2 "Resistor_SMD:R_0603_1608Metric" V 4680 4540 50  0001 C CNN
 F 3 "~" H 4750 4540 50  0001 C CNN
 	1    4750 4540
@@
 F 0 "IC13" H 6100 5040 50  0000 C CNN
 F 1 "INA199A1DCKT_v2" H 6370 4950 50  0000 C CNN
-F 2 "SOT65P210X110-6N" H 7120 4480 50  0001 L CNN
+F 2 "Package_TO_SOT_SMD:SOT-363_SC-70-6" H 7120 4480 50  0001 L CNN
 F 3 "http://www.ti.com/lit/gpn/INA199" H 7120 4380 50  0001 L CNN
 F 4 "26V, bi-directional, zero-drift, low-/high-side, voltage output current sense amplifier" H 7120 4280 50  0001 L CNN "Description"
@@
 F 0 "C25" H 6485 3336 50  0000 L CNN
 F 1 "0.1u" H 6485 3245 50  0000 L CNN
-F 2 "" H 6408 3140 50  0001 C CNN
+F 2 "Capacitor_SMD:C_0603_1608Metric" H 6408 3140 50  0001 C CNN
 F 3 "~" H 6370 3290 50  0001 C CNN
 	1    6370 3290
