File: rsp02_LoadSW_OCP_Circuit_v1_2.sch (KiCad schematic (older format))
At the start: 26 parts, among them IC1 OP291GSZ_v2, J1 Conn_01x02, J2 Conn_01x04, J3 Conn_01x02, J4 Conn_01x02, Q1 SISS23DN-T1-GE3, Q2 IRF7404, Q3 BC848B

Commit message: Changed Design plan(Module Design)
Parts:
- removed C1, C2, C3: 0.1u, Capacitor_SMD:C_0402_1005Metric, symbol Device:C
- removed CR1, CR2, CR3, CR4: 1SS352_H3FT, mypartsLib:1SS352_H3FT, symbol mypartsLib:1SS352_H3FT
- removed IC1: OP291GSZ_v2, Package_SO:SOIC-8_3.9x4.9mm_P1.27mm, symbol mypartsLib:OP291GSZ_v2
- removed J1, J3, J4: Conn_01x02, Connector_PinHeader_2.00mm:PinHeader_1x02_P2.00mm_Vertical, symbol Connector_Generic:Conn_01x02
- removed J2: Conn_01x04, Connector_PinHeader_2.00mm:PinHeader_1x04_P2.00mm_Vertical, symbol Connector_Generic:Conn_01x04
- removed Q1: SISS23DN-T1-GE3, mypartsLib:POWERPAK-1212-8, symbol mypartsLib:SISS23DN-T1-GE3
- removed Q2: IRF7404, Package_SO:SOIC-8_3.9x4.9mm_P1.27mm, symbol Transistor_FET:IRF7404
- removed Q3: BC848B, Package_TO_SOT_SMD:SOT-23, symbol mypartsLib:BC848B
- removed R1, R6, R8, Rh1: 100k, Resistor_SMD:R_0402_1005Metric, symbol Device:R
- removed R2: 0.5, Resistor_SMD:R_2512_6332Metric, symbol Device:R
- removed R3: 1000k, Resistor_SMD:R_0402_1005Metric, symbol Device:R
- removed R4, R7: 10k, Resistor_SMD:R_0402_1005Metric, symbol Device:R
- removed R5: 1k, Resistor_SMD:R_0402_1005Metric, symbol Device:R
- removed RV1, RV2: 100k, Potentiometer_SMD:Potentiometer_Bourns_3314G_Vertical, symbol Device:R_Potentiometer_Trim
Connections:
- no-connect marks 5 -> 0
Other:
- note added: "3.3V Output"
- note added: "3V Output"
- note added: "5V Output"

Commit message: Update
Parts:
- added J1, J10, J11, J12, J13, J14, J2, J3, J4, J5, J6, J7, J8, J9: Conn_01x02, symbol Connector_Generic:Conn_01x02
- added J15, J16: Conn_01x10, symbol Connector_Generic:Conn_01x10
- added R1, R10, R11, R12, R13, R14, R15, R16, R17, R18, R19, R2, R3, R4, R5, R6, R7, R8, R9: 0, symbol Device:R_Small
Connections:
- net GNDA: now also J1.1 (Pin_1), J10.2 (Pin_2), J11.2 (Pin_2), J12.2 (Pin_2), J13.2 (Pin_2), J14.2 (Pin_2), J15.1 (Pin_1), J16.1 (Pin_1), J2.1 (Pin_1), J3.1 (Pin_1), J4.2 (Pin_2), J5.2 (Pin_2), J6.2 (Pin_2), J7.2 (Pin_2), J8.2 (Pin_2), J9.2 (Pin_2)
- net LoadSW_OCP_Attitude/LSWE1: now also R14.1
- net LoadSW_OCP_Attitude/LSWE2: now also R15.1
- net LoadSW_OCP_C&DH OBC/LSWE1: now also R12.1
- net LoadSW_OCP_C&DH OBC/LSWE2: now also R13.1
- net LoadSW_OCP_Deployment Cover/LSWE1: now also R16.1
- net LoadSW_OCP_Deployment Cover/LSWE2: now also R17.1
- net LoadSW_OCP_Mission OBC/LSWE1: now also R10.1
- net LoadSW_OCP_Mission OBC/LSWE2: now also R11.1
- net LoadSW_OCP_Nichrome Wire/LSWE1: now also R18.1
- net LoadSW_OCP_Nichrome Wire/LSWE2: now also R19.1
- net LoadSW_OCP_RX/LSWE1: now also R8.1
- net LoadSW_OCP_RX/LSWE2: now also R9.1
- net LoadSW_OCP_TX PA/LSWE1: now also R4.1
- net LoadSW_OCP_TX PA/LSWE2: now also R5.1
- net LoadSW_OCP_TX/LSWE1: now also R6.1
- net LoadSW_OCP_TX/LSWE2: now also R7.1
- net Power_Attitude: now also J12.1 (Pin_1)
- net Power_C&DH: now also J11.1 (Pin_1)
- net Power_DeploymentCover: now also J13.1 (Pin_1)
- net Power_IN_3_0V: now also J3.2 (Pin_2), R3.1
- net Power_IN_3_3V: now also J2.2 (Pin_2), R2.1
- net Power_IN_5_0V: now also J1.2 (Pin_2), R1.1
- net Power_Mission: now also J10.1 (Pin_1)
- net Power_NichromeWire: now also J14.1 (Pin_1)
- net Power_RX: now also J9.1 (Pin_1)
- net Power_TX: now also J8.1 (Pin_1)
- net Power_TX_PA: now also J7.1 (Pin_1)
- new net ASWE_fromIOE: J16.7 (Pin_7), R14.2
- new net DCSWE_fromIOE: J16.6 (Pin_6), R16.2
- new net Imon_Attde: J15.5 (Pin_5)
- new net Imon_CDH: J15.6 (Pin_6)
- new net Imon_DplyCvr: J15.4 (Pin_4)
- new net Imon_Mission: J15.7 (Pin_7)
- new net Imon_NicWire: J15.3 (Pin_3)
- new net Imon_TX: J15.8 (Pin_8), J15.9 (Pin_9)
- new net Imon_TXPA: J15.10 (Pin_10)
- new net MSWE_fromIOE: J16.8 (Pin_8), R10.2
- new net NWSWE_fromIOE: J16.5 (Pin_5), R18.2
- new net NWSWE_fromRX: J16.2 (Pin_2), R19.2
- new net Power_Line_3_0V_DplyCvr: R17.2
- new net Power_Line_3_3V_A: R15.2
- new net Power_Line_3_3V_C: R12.2, R13.2
- new net Power_Line_3_3V_M: R11.2
- new net Power_Line_3_3V_RX: R8.2, R9.2
- new net Power_Line_5_0V_TXPA: R5.2
- new net Power_Mon_3_0V: J6.1 (Pin_1), R3.2
- new net Power_Mon_3_3V: J5.1 (Pin_1), R2.2
- new net Power_Mon_5_0V: J4.1 (Pin_1), R1.2
- new net TPASWE_fromIOE: J16.10 (Pin_10), R4.2
- new net TXSWE_fromIOE: J16.9 (Pin_9), R6.2
- new net TXSWE_fromRX: J16.3 (Pin_3), R7.2
- no-connect marks 0 -> 2
Other:
- note added: "3.0V Input"
- note added: "3.0V Output"
- note added: "3.3V Input"
- note added: "5.0V Input"
- note added: "5.0V Output"
- note added: "LoadSW Deactive"
- note added: "OCP : \nDeactive"
- note added: "SW Control from RX"
- note added: "[High Active]"
- note removed: "3V Output"
- note removed: "5V Output"

Commit message: Update PCB
Parts:
- J1, J10, J11, J12, J13, J14, J2, J3, J4, J5, J6, J7, J8, J9: footprint (none) -> TerminalBlock_Phoenix:TerminalBlock_Phoenix_MKDS-3-2-5.08_1x02_P5.08mm_Horizontal
- J15, J16: footprint (none) -> TerminalBlock_Phoenix:TerminalBlock_Phoenix_MKDS-3-10-5.08_1x10_P5.08mm_Horizontal
- R1, R10, R11, R12, R13, R14, R15, R16, R17, R18, R19, R2, R3, R4, R5, R6, R7, R8, R9: footprint (none) -> Resistor_SMD:R_0603_1608Metric
Other:
- moved on the sheet: J15, J16

Commit message: PCB Update
Parts:
- J4, J5, J6: footprint TerminalBlock_Phoenix:TerminalBlock_Phoenix_MKDS-3-2-5.08_1x02_P5.08mm_Horizontal -> Connector_PinHeader_2.54mm:PinHeader_1x02_P2.54mm_Vertical
Connections:
- net GNDA: now also J1.2 (Pin_2), J2.2 (Pin_2), J3.2 (Pin_2); no longer J1.1 (Pin_1), J2.1 (Pin_1), J3.1 (Pin_1)
- net Power_IN_3_0V: now also J3.1 (Pin_1); no longer J3.2 (Pin_2)
- net Power_IN_3_3V: now also J2.1 (Pin_1); no longer J2.2 (Pin_2)
- net Power_IN_5_0V: now also J1.1 (Pin_1); no longer J1.2 (Pin_2)
Changed lines of the file:
@@
 L Connector_Generic:Conn_01x02 J1
 U 1 1 5FFB79CD
-P 1040 850
-F 0 "J1" H 958 525 50  0000 C CNN
-F 1 "Conn_01x02" H 958 616 50  0000 C CNN
-F 2 "TerminalBlock_Phoenix:TerminalBlock_Phoenix_MKDS-3-2-5.08_1x02_P5.08mm_Horizontal" H 1040 850 50  0001 C CNN
-F 3 "~" H 1040 850 50  0001 C CNN
-	1    1040 850
-	-1   0    0    1
+P 1040 750
+F 0 "J1" H 1160 700 50  0000 C CNN
+F 1 "Conn_01x02" H 958 516 50  0000 C CNN
+F 2 "TerminalBlock_Phoenix:TerminalBlock_Phoenix_MKDS-3-2-5.08_1x02_P5.08mm_Horizontal" H 1040 750 50  0001 C CNN
+F 3 "~" H 1040 750 50  0001 C CNN
+	1    1040 750
+	-1   0    0    -1
 $EndComp
 $Comp
 L Connector_Generic:Conn_01x02 J2
 U 1 1 5FFB967E
-P 1050 1300
-F 0 "J2" H 968 975 50  0000 C CNN
-F 1 "Conn_01x02" H 968 1066 50  0000 C CNN
-F 2 "TerminalBlock_Phoenix:TerminalBlock_Phoenix_MKDS-3-2-5.08_1x02_P5.08mm_Horizontal" H 1050 1300 50  0001 C CNN
-F 3 "~" H 1050 1300 50  0001 C CNN
-	1    1050 1300
-	-1   0    0    1
+P 1050 1200
+F 0 "J2" H 1180 1150 50  0000 C CNN
+F 1 "Conn_01x02" H 968 966 50  0000 C CNN
+F 2 "TerminalBlock_Phoenix:TerminalBlock_Phoenix_MKDS-3-2-5.08_1x02_P5.08mm_Horizontal" H 1050 1200 50  0001 C CNN
+F 3 "~" H 1050 1200 50  0001 C CNN
+	1    1050 1200
+	-1   0    0    -1
 $EndComp
 $Comp
 L Connector_Generic:Conn_01x02 J3
 U 1 1 5FFBA725
-P 1050 1750
-F 0 "J3" H 968 1425 50  0000 C CNN
-F 1 "Conn_01x02" H 968 1516 50  0000 C CNN
-F 2 "TerminalBlock_Phoenix:TerminalBlock_Phoenix_MKDS-3-2-5.08_1x02_P5.08mm_Horizontal" H 1050 1750 50  0001 C CNN
-F 3 "~" H 1050 1750 50  0001 C CNN
-	1    1050 1750
-	-1   0    0    1
+P 1050 1650
+F 0 "J3" H 1190 1590 50  0000 C CNN
+F 1 "Conn_01x02" H 968 1416 50  0000 C CNN
+F 2 "TerminalBlock_Phoenix:TerminalBlock_Phoenix_MKDS-3-2-5.08_1x02_P5.08mm_Horizontal" H 1050 1650 50  0001 C CNN
+F 3 "~" H 1050 1650 50  0001 C CNN
+	1    1050 1650
+	-1   0    0    -1
 $EndComp
 $Comp
@@
 F 0 "J4" H 1930 2142 50  0000 L CNN
 F 1 "Conn_01x02" H 1930 2051 50  0000 L CNN
-F 2 "TerminalBlock_Phoenix:TerminalBlock_Phoenix_MKDS-3-2-5.08_1x02_P5.08mm_Horizontal" H 1850 2150 50  0001 C CNN
+F 2 "Connector_PinHeader_2.54mm:PinHeader_1x02_P2.54mm_Vertical" H 1850 2150 50  0001 C CNN
 F 3 "~" H 1850 2150 50  0001 C CNN
 	1    1850 2150
@@
 F 0 "J5" H 1930 2472 50  0000 L CNN
 F 1 "Conn_01x02" H 1930 2381 50  0000 L CNN
-F 2 "TerminalBlock_Phoenix:TerminalBlock_Phoenix_MKDS-3-2-5.08_1x02_P5.08mm_Horizontal" H 1850 2480 50  0001 C CNN
+F 2 "Connector_PinHeader_2.54mm:PinHeader_1x02_P2.54mm_Vertical" H 1850 2480 50  0001 C CNN
 F 3 "~" H 1850 2480 50  0001 C CNN
 	1    1850 2480
@@
 F 0 "J6" H 1930 2872 50  0000 L CNN
 F 1 "Conn_01x02" H 1930 2781 50  0000 L CNN
-F 2 "TerminalBlock_Phoenix:TerminalBlock_Phoenix_MKDS-3-2-5.08_1x02_P5.08mm_Horizontal" H 1850 2880 50  0001 C CNN
+F 2 "Connector_PinHeader_2.54mm:PinHeader_1x02_P2.54mm_Vertical" H 1850 2880 50  0001 C CNN
 F 3 "~" H 1850 2880 50  0001 C CNN
 	1    1850 2880

Commit message: PCB Update
Parts:
- J15: footprint TerminalBlock_Phoenix:TerminalBlock_Phoenix_MKDS-3-10-5.08_1x10_P5.08mm_Horizontal -> Connector_PinHeader_2.54mm:PinHeader_1x10_P2.54mm_Vertical
Connections:
- net Imon_TX: no longer J15.8 (Pin_8)
- new net Imon_RX: J15.8 (Pin_8)
Changed lines of the file:
@@
 	5600 1700 5400 1700
 Text GLabel 5600 2400 2    39   Output ~ 0
-Imon_TX
+Imon_RX
 Wire Wire Line
 	5410 2400 5600 2400
@@
 F 0 "J15" H 4180 7470 50  0000 C CNN
 F 1 "Conn_01x10" H 4370 7570 50  0000 C CNN
-F 2 "TerminalBlock_Phoenix:TerminalBlock_Phoenix_MKDS-3-10-5.08_1x10_P5.08mm_Horizontal" H 4050 7150 50  0001 C CNN
+F 2 "Connector_PinHeader_2.54mm:PinHeader_1x10_P2.54mm_Vertical" H 4050 7150 50  0001 C CNN
 F 3 "~" H 4050 7150 50  0001 C CNN
 	1    4050 7150
@@
 Imon_TX
 Text GLabel 3700 6850 0    39   Input ~ 0
-Imon_TX
+Imon_RX
 Text GLabel 3700 6950 0    39   Input ~ 0
 Imon_Mission

Commit message: PCB Design Finished
Connections:
- net Power_Line_3_0V_DplyCvr: no longer R17.2
- net Power_Line_3_3V_A: no longer R15.2
- net Power_Line_3_3V_M: no longer R11.2
- net Power_Line_5_0V_TXPA: no longer R5.2
- no-connect marks 2 -> 6
Changed lines of the file:
@@
 Wire Wire Line
 	7240 1000 7500 1000
-Wire Wire Line
-	6900 1000 6900 800
-Wire Wire Line
-	6900 1000 7040 1000
 Connection ~ 6900 800
 Wire Wire Line
@@
 Wire Wire Line
 	7240 3100 7500 3100
-Wire Wire Line
-	6900 2900 6900 3100
-Wire Wire Line
-	6900 3100 7040 3100
 Connection ~ 6900 2900
 Wire Wire Line
@@
 $EndComp
 Wire Wire Line
-	7040 4500 6900 4500
-Wire Wire Line
 	7240 4500 7500 4500
-Wire Wire Line
-	6900 4500 6900 4300
 Connection ~ 6900 4300
 Wire Wire Line
@@
 Wire Wire Line
 	7240 5200 7500 5200
-Wire Wire Line
-	6900 5200 6900 5000
-Wire Wire Line
-	7040 5200 6900 5200
-Connection ~ 6900 5000
-Wire Wire Line
-	6900 5000 7500 5000
 Wire Wire Line
 	6790 5100 7040 5100
@@
 Text Notes 6660 6020 2    39   ~ 0
 [High Active]
-Wire Wire Line
-	5410 5000 6900 5000
 Wire Wire Line
 	5400 4300 6900 4300
@@
 Wire Wire Line
 	5400 5700 7500 5700
+NoConn ~ 7040 3100
+NoConn ~ 7040 4500
+Wire Wire Line
+	5410 5000 7500 5000
+NoConn ~ 7040 5200
+NoConn ~ 7040 1000
 $EndSCHEMATC
