File: rsp02_module_CS_3_3V.sch (KiCad schematic (older format))
At the start: 5 parts, among them IC14 INA199A1DCKT_v2

Commit message: Update PCB
Parts:
- C26: footprint (none) -> Capacitor_SMD:C_0603_1608Metric
- IC14: footprint SOT65P210X110-6N -> Package_TO_SOT_SMD:SOT-363_SC-70-6
- R115, R116: footprint (none) -> Resistor_SMD:R_0603_1608Metric
- R117: footprint (none) -> Resistor_SMD:R_2512_6332Metric
Changed lines of the file:
@@
 $Descr A4 11693 8268
 encoding utf-8
-Sheet 17 17
+Sheet 10 17
 Title "rsp02_module_Current Sense_3_3V"
 Date "2020-12-07"
@@
 AR Path="/5FD18C31/5FD0FFD7" Ref="R108"  Part="1"
 AR Path="/5FD18BF5/5FD0FFD7" Ref="R111"  Part="1"
-F 0 "R117" V 5490 2500 50  0000 C CNN
+F 0 "R96" V 5490 2500 50  0000 C CNN
 F 1 "0.02" V 5660 2500 50  0000 C CNN
-F 2 "" V 5500 2500 50  0001 C CNN
+F 2 "Resistor_SMD:R_2512_6332Metric" V 5500 2500 50  0001 C CNN
 F 3 "~" H 5570 2500 50  0001 C CNN
 	1    5570 2500
@@
 AR Path="/5FD18C31/5FCF83F6" Ref="R106"  Part="1"
 AR Path="/5FD18BF5/5FCF83F6" Ref="R109"  Part="1"
-F 0 "R115" V 4830 4450 50  0000 C CNN
+F 0 "R94" V 4830 4450 50  0000 C CNN
 F 1 "0" V 4750 4340 50  0000 C CNN
-F 2 "" V 4680 4340 50  0001 C CNN
+F 2 "Resistor_SMD:R_0603_1608Metric" V 4680 4340 50  0001 C CNN
 F 3 "~" H 4750 4340 50  0001 C CNN
 	1    4750 4340
@@
 AR Path="/5FD18C31/5FCF83F7" Ref="R107"  Part="1"
 AR Path="/5FD18BF5/5FCF83F7" Ref="R110"  Part="1"
-F 0 "R116" V 4840 4640 50  0000 C CNN
+F 0 "R95" V 4840 4640 50  0000 C CNN
 F 1 "0" V 4750 4540 50  0000 C CNN
-F 2 "" V 4680 4540 50  0001 C CNN
+F 2 "Resistor_SMD:R_0603_1608Metric" V 4680 4540 50  0001 C CNN
 F 3 "~" H 4750 4540 50  0001 C CNN
 	1    4750 4540
@@
 AR Path="/5FD18C31/5FCF83F8" Ref="IC11"  Part="1"
 AR Path="/5FD18BF5/5FCF83F8" Ref="IC12"  Part="1"
-F 0 "IC14" H 6100 5040 50  0000 C CNN
+F 0 "IC7" H 6100 5040 50  0000 C CNN
 F 1 "INA199A1DCKT_v2" H 6370 4950 50  0000 C CNN
-F 2 "SOT65P210X110-6N" H 7120 4480 50  0001 L CNN
+F 2 "Package_TO_SOT_SMD:SOT-363_SC-70-6" H 7120 4480 50  0001 L CNN
 F 3 "http://www.ti.com/lit/gpn/INA199" H 7120 4380 50  0001 L CNN
 F 4 "26V, bi-directional, zero-drift, low-/high-side, voltage output current sense amplifier" H 7120 4280 50  0001 L CNN "Description"
@@
 AR Path="/5FD18C31/5FD23316" Ref="C23"  Part="1"
 AR Path="/5FD18BF5/5FD23316" Ref="C24"  Part="1"
-F 0 "C26" H 6485 3336 50  0000 L CNN
+F 0 "C19" H 6485 3336 50  0000 L CNN
 F 1 "0.1u" H 6485 3245 50  0000 L CNN
-F 2 "" H 6408 3140 50  0001 C CNN
+F 2 "Capacitor_SMD:C_0603_1608Metric" H 6408 3140 50  0001 C CNN
 F 3 "~" H 6370 3290 50  0001 C CNN
 	1    6370 3290

Commit message: PCB Update
Changed lines of the file:
@@
 $Descr A4 11693 8268
 encoding utf-8
-Sheet 10 17
+Sheet 15 17
 Title "rsp02_module_Current Sense_3_3V"
 Date "2020-12-07"
@@
 AR Path="/5FD18C31/5FD0FFD7" Ref="R108"  Part="1"
 AR Path="/5FD18BF5/5FD0FFD7" Ref="R111"  Part="1"
-F 0 "R96" V 5490 2500 50  0000 C CNN
+F 0 "R111" V 5490 2500 50  0000 C CNN
 F 1 "0.02" V 5660 2500 50  0000 C CNN
 F 2 "Resistor_SMD:R_2512_6332Metric" V 5500 2500 50  0001 C CNN
@@
 AR Path="/5FD18C31/5FCF83F6" Ref="R106"  Part="1"
 AR Path="/5FD18BF5/5FCF83F6" Ref="R109"  Part="1"
-F 0 "R94" V 4830 4450 50  0000 C CNN
+F 0 "R109" V 4830 4450 50  0000 C CNN
 F 1 "0" V 4750 4340 50  0000 C CNN
 F 2 "Resistor_SMD:R_0603_1608Metric" V 4680 4340 50  0001 C CNN
@@
 AR Path="/5FD18C31/5FCF83F7" Ref="R107"  Part="1"
 AR Path="/5FD18BF5/5FCF83F7" Ref="R110"  Part="1"
-F 0 "R95" V 4840 4640 50  0000 C CNN
+F 0 "R110" V 4840 4640 50  0000 C CNN
 F 1 "0" V 4750 4540 50  0000 C CNN
 F 2 "Resistor_SMD:R_0603_1608Metric" V 4680 4540 50  0001 C CNN
@@
 AR Path="/5FD18C31/5FCF83F8" Ref="IC11"  Part="1"
 AR Path="/5FD18BF5/5FCF83F8" Ref="IC12"  Part="1"
-F 0 "IC7" H 6100 5040 50  0000 C CNN
+F 0 "IC12" H 6100 5040 50  0000 C CNN
 F 1 "INA199A1DCKT_v2" H 6370 4950 50  0000 C CNN
 F 2 "Package_TO_SOT_SMD:SOT-363_SC-70-6" H 7120 4480 50  0001 L CNN
@@
 AR Path="/5FD18C31/5FD23316" Ref="C23"  Part="1"
 AR Path="/5FD18BF5/5FD23316" Ref="C24"  Part="1"
-F 0 "C19" H 6485 3336 50  0000 L CNN
+F 0 "C24" H 6485 3336 50  0000 L CNN
 F 1 "0.1u" H 6485 3245 50  0000 L CNN
 F 2 "Capacitor_SMD:C_0603_1608Metric" H 6408 3140 50  0001 C CNN

Commit message: PCB Design Finished
Changed lines of the file:
@@
 $Descr A4 11693 8268
 encoding utf-8
-Sheet 15 17
+Sheet 11 17
 Title "rsp02_module_Current Sense_3_3V"
 Date "2020-12-07"
@@
 AR Path="/5FD18C31/5FD0FFD7" Ref="R108"  Part="1"
 AR Path="/5FD18BF5/5FD0FFD7" Ref="R111"  Part="1"
-F 0 "R111" V 5490 2500 50  0000 C CNN
+F 0 "R117" V 5490 2500 50  0000 C CNN
 F 1 "0.02" V 5660 2500 50  0000 C CNN
 F 2 "Resistor_SMD:R_2512_6332Metric" V 5500 2500 50  0001 C CNN
@@
 AR Path="/5FD18C31/5FCF83F6" Ref="R106"  Part="1"
 AR Path="/5FD18BF5/5FCF83F6" Ref="R109"  Part="1"
-F 0 "R109" V 4830 4450 50  0000 C CNN
+F 0 "R115" V 4830 4450 50  0000 C CNN
 F 1 "0" V 4750 4340 50  0000 C CNN
 F 2 "Resistor_SMD:R_0603_1608Metric" V 4680 4340 50  0001 C CNN
@@
 AR Path="/5FD18C31/5FCF83F7" Ref="R107"  Part="1"
 AR Path="/5FD18BF5/5FCF83F7" Ref="R110"  Part="1"
-F 0 "R110" V 4840 4640 50  0000 C CNN
+F 0 "R116" V 4840 4640 50  0000 C CNN
 F 1 "0" V 4750 4540 50  0000 C CNN
 F 2 "Resistor_SMD:R_0603_1608Metric" V 4680 4540 50  0001 C CNN
@@
 AR Path="/5FD18C31/5FCF83F8" Ref="IC11"  Part="1"
 AR Path="/5FD18BF5/5FCF83F8" Ref="IC12"  Part="1"
-F 0 "IC12" H 6100 5040 50  0000 C CNN
+F 0 "IC14" H 6100 5040 50  0000 C CNN
 F 1 "INA199A1DCKT_v2" H 6370 4950 50  0000 C CNN
 F 2 "Package_TO_SOT_SMD:SOT-363_SC-70-6" H 7120 4480 50  0001 L CNN
@@
 AR Path="/5FD18C31/5FD23316" Ref="C23"  Part="1"
 AR Path="/5FD18BF5/5FD23316" Ref="C24"  Part="1"
-F 0 "C24" H 6485 3336 50  0000 L CNN
+F 0 "C26" H 6485 3336 50  0000 L CNN
 F 1 "0.1u" H 6485 3245 50  0000 L CNN
 F 2 "Capacitor_SMD:C_0603_1608Metric" H 6408 3140 50  0001 C CNN
