File: rsp02_module_LoadSW_noOCP.sch (KiCad schematic (older format))
At the start: 23 parts, among them IC1 OP291GSZ_v2, Q1 SISS23DN-T1-GE3, Q2 IRF7404, Q3 BC848B

Commit message: Update
Parts:
- removed C1: 0.1u, Capacitor_SMD:C_0402_1005Metric, symbol Device:C
- removed CR1, CR2: 1SS352_H3FT, mypartsLib:1SS352_H3FT, symbol mypartsLib:1SS352_H3FT
- removed IC1: OP291GSZ_v2, Package_SO:SOIC-8_3.9x4.9mm_P1.27mm, symbol mypartsLib:OP291GSZ_v2
- removed Q1: SISS23DN-T1-GE3, mypartsLib:POWERPAK-1212-8, symbol mypartsLib:SISS23DN-T1-GE3
- removed Q3: BC848B, Package_TO_SOT_SMD:SOT-23, symbol mypartsLib:BC848B
- removed R1, R6, R8: 100k, Resistor_SMD:R_0402_1005Metric, symbol Device:R
- removed R7, R9: 10k, Resistor_SMD:R_0402_1005Metric, symbol Device:R
- removed RV1: 100k, Potentiometer_SMD:Potentiometer_Bourns_3314G_Vertical, symbol Device:R_Potentiometer_Trim
- added C22: 0.1u, Capacitor_SMD:C_0402_1005Metric, symbol Device:C
- added CR29, CR30: 1SS352_H3FT, mypartsLib:1SS352_H3FT, symbol mypartsLib:1SS352_H3FT
- added IC8: OP291GSZ_v2, Package_SO:SOIC-8_3.9x4.9mm_P1.27mm, symbol mypartsLib:OP291GSZ_v2
- added Q22: SISS23DN-T1-GE3, mypartsLib:POWERPAK-1212-8, symbol mypartsLib:SISS23DN-T1-GE3
- added Q24: BC848B, Package_TO_SOT_SMD:SOT-23, symbol mypartsLib:BC848B
- added R83, R88, R91: 100k, Resistor_SMD:R_0402_1005Metric, symbol Device:R
- added R89, R90: 10k, Resistor_SMD:R_0402_1005Metric, symbol Device:R
- added RV15: 100k, Potentiometer_SMD:Potentiometer_Bourns_3314G_Vertical, symbol Device:R_Potentiometer_Trim
- renumbered C2 to C23, C3 to C24, CR3 to CR31, CR4 to CR32, Q2 to Q23, R2 to R84, R3 to R85, R4 to R86, R5 to R87, RV2 to RV16, Rh1 to Rh8
Connections:
- net GND: now also C22.2, IC8.4 (-V), Q24.2 (emitter), R83.2, R90.2
- net INPUT: now also IC8.8 (+V), R91.1, RV15.1, RV15.2
- net OUTPUT: now also Q22.5 (D(1)), Q22.6 (D(2)), Q22.7 (D(3)), Q22.8 (D(4))
- net at R85.1, RV16.3: now also C22.1, CR29.2 (anode), IC8.2 (-INA)
- net at R84.1, RV16.1, RV16.2: now also CR29.1 (cathode), Q22.1 (S(1)), Q22.2 (S(2)), Q22.3 (S(3)), R88.1
- net at Q23.5 (D), Q23.6 (D), Q23.7 (D)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: now also CR30.1 (cathode)
- net at R86.2, Rh8.1: now also CR30.2 (anode), IC8.1 (OUTA)
- net at Rh8.2: now also IC8.3 (+INA), R83.1, RV15.3
- net at Q23.1 (S), Q23.2 (S), Q23.3 (S): now also Q22.4 (G), R88.2
- net at Q23.4 (G): now also Q24.3 (collector), R91.2
- net at CR31.1 (cathode), CR32.1 (cathode): now also R89.2
- new net: Q24.1 (base), R89.1, R90.1

Commit message: Update Design
Parts:
- removed C22, C23, C24: 0.1u, Capacitor_SMD:C_0402_1005Metric, symbol Device:C
- removed CR29, CR30, CR31, CR32: 1SS352_H3FT, mypartsLib:1SS352_H3FT, symbol mypartsLib:1SS352_H3FT
- removed IC8: OP291GSZ_v2, Package_SO:SOIC-8_3.9x4.9mm_P1.27mm, symbol mypartsLib:OP291GSZ_v2
- removed R83, R88, Rh8: 100k, Resistor_SMD:R_0402_1005Metric, symbol Device:R
- removed R84: 0.5, Resistor_SMD:R_2512_6332Metric, symbol Device:R
- removed R85: 1000k, Resistor_SMD:R_0402_1005Metric, symbol Device:R
- removed R86, R89: 10k, Resistor_SMD:R_0402_1005Metric, symbol Device:R
- removed R87: 1k, Resistor_SMD:R_0402_1005Metric, symbol Device:R
- removed RV15, RV16: 100k, Potentiometer_SMD:Potentiometer_Bourns_3314G_Vertical, symbol Device:R_Potentiometer_Trim
- added CR27, CR28: 1SS352_H3FT, mypartsLib:1SS352_H3FT, symbol mypartsLib:1SS352_H3FT
- added R92: 10k, Resistor_SMD:R_0402_1005Metric, symbol Device:R
- added R93: 100k, Resistor_SMD:R_0402_1005Metric, symbol Device:R
- R90: value 10k -> 100k
- R91: value 100k -> 10k
Connections:
- net GND: now also Q23.5 (D), Q23.6 (D), Q23.7 (D), Q23.8 (D), R92.2; no longer R90.2
- net INPUT: now also Q22.1 (S(1)), Q22.2 (S(2)), Q22.3 (S(3)), R90.1, R93.1; no longer R91.1
- net LSWE1: now also CR27.2 (anode)
- net LSWE2: now also CR28.2 (anode)
- net at Q22.4 (G), Q23.1 (S), Q23.2 (S)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: now also R90.2
- net at Q23.4 (G), Q24.3 (collector): now also R93.2; no longer R91.2
- net at Q24.1 (base): now also R91.1, R92.1; no longer R90.1
- new net: CR27.1 (cathode), CR28.1 (cathode), R91.2
- no-connect marks 3 -> 0

Commit message: Update PCB
Parts:
- R90, R91, R92, R93: footprint Resistor_SMD:R_0402_1005Metric -> Resistor_SMD:R_0603_1608Metric
Changed lines of the file:
@@
 F 0 "R90" H 7000 1750 50  0000 L CNN
 F 1 "100k" H 7000 1550 50  0000 L CNN
-F 2 "Resistor_SMD:R_0402_1005Metric" V 6880 1650 50  0001 C CNN
+F 2 "Resistor_SMD:R_0603_1608Metric" V 6880 1650 50  0001 C CNN
 F 3 "~" H 6950 1650 50  0001 C CNN
 	1    6950 1650
@@
 F 0 "R93" H 9300 2250 50  0000 L CNN
 F 1 "100k" H 9300 2050 50  0000 L CNN
-F 2 "Resistor_SMD:R_0402_1005Metric" V 9180 2150 50  0001 C CNN
+F 2 "Resistor_SMD:R_0603_1608Metric" V 9180 2150 50  0001 C CNN
 F 3 "~" H 9250 2150 50  0001 C CNN
 	1    9250 2150
@@
 F 0 "R92" H 8850 5000 50  0000 L CNN
 F 1 "10k" H 8850 4800 50  0000 L CNN
-F 2 "Resistor_SMD:R_0402_1005Metric" V 8730 4900 50  0001 C CNN
+F 2 "Resistor_SMD:R_0603_1608Metric" V 8730 4900 50  0001 C CNN
 F 3 "~" H 8800 4900 50  0001 C CNN
 	1    8800 4900
@@
 F 0 "R91" V 8600 4550 50  0000 L CNN
 F 1 "10k" V 8400 4550 50  0000 L CNN
-F 2 "Resistor_SMD:R_0402_1005Metric" V 8430 4600 50  0001 C CNN
+F 2 "Resistor_SMD:R_0603_1608Metric" V 8430 4600 50  0001 C CNN
 F 3 "~" H 8500 4600 50  0001 C CNN
 	1    8500 4600

Commit message: PCB Update
Changed lines of the file:
@@
 $Descr A4 11693 8268
 encoding utf-8
-Sheet 9 17
+Sheet 6 17
 Title "rsp02_module_LoadSW_OCP_noOCP"
 Date "2020-12-07"
@@
 AR Path="/5FD193EF/5FD0BC5C" Ref="Q22"  Part="1"
 AR Path="/5FD18D34/5FD0BC5C" Ref="Q13"  Part="1"
-F 0 "Q22" H 7900 1617 50  0000 C CNN
+F 0 "Q13" H 7900 1617 50  0000 C CNN
 F 1 "SISS23DN-T1-GE3" H 7900 1526 50  0000 C CNN
 F 2 "mypartsLib:POWERPAK-1212-8" H 7900 800 50  0001 C CNN
@@
 AR Path="/5FD193EF/5FD0BC5D" Ref="R90"  Part="1"
 AR Path="/5FD18D34/5FD0BC5D" Ref="R64"  Part="1"
-F 0 "R90" H 7000 1750 50  0000 L CNN
+F 0 "R64" H 7000 1750 50  0000 L CNN
 F 1 "100k" H 7000 1550 50  0000 L CNN
 F 2 "Resistor_SMD:R_0603_1608Metric" V 6880 1650 50  0001 C CNN
@@
 AR Path="/5FD193EF/5FD0BC5E" Ref="R93"  Part="1"
 AR Path="/5FD18D34/5FD0BC5E" Ref="R67"  Part="1"
-F 0 "R93" H 9300 2250 50  0000 L CNN
+F 0 "R67" H 9300 2250 50  0000 L CNN
 F 1 "100k" H 9300 2050 50  0000 L CNN
 F 2 "Resistor_SMD:R_0603_1608Metric" V 9180 2150 50  0001 C CNN
@@
 AR Path="/5FD193EF/5FD0BC5F" Ref="R92"  Part="1"
 AR Path="/5FD18D34/5FD0BC5F" Ref="R66"  Part="1"
-F 0 "R92" H 8850 5000 50  0000 L CNN
+F 0 "R66" H 8850 5000 50  0000 L CNN
 F 1 "10k" H 8850 4800 50  0000 L CNN
 F 2 "Resistor_SMD:R_0603_1608Metric" V 8730 4900 50  0001 C CNN
@@
 AR Path="/5FD193EF/5FD2B5CE" Ref="Q24"  Part="1"
 AR Path="/5FD18D34/5FD2B5CE" Ref="Q15"  Part="1"
-F 0 "Q24" H 9294 4646 50  0000 L CNN
+F 0 "Q15" H 9294 4646 50  0000 L CNN
 F 1 "BC848B" H 9294 4555 50  0000 L CNN
 F 2 "Package_TO_SOT_SMD:SOT-23" H 8950 5100 50  0001 L CNN
@@
 AR Path="/5FD193EF/5FD2B5CD" Ref="Q23"  Part="1"
 AR Path="/5FD18D34/5FD2B5CD" Ref="Q14"  Part="1"
-F 0 "Q23" H 7705 2404 50  0000 L CNN
+F 0 "Q14" H 7705 2404 50  0000 L CNN
 F 1 "IRF7404" H 7705 2495 50  0000 L CNN
 F 2 "Package_SO:SOIC-8_3.9x4.9mm_P1.27mm" H 7700 2375 50  0001 L CIN
@@
 AR Path="/5FD193EF/5FD2B5CF" Ref="CR28"  Part="1"
 AR Path="/5FD18D34/5FD2B5CF" Ref="CR18"  Part="1"
-F 0 "CR28" H 7700 4700 50  0000 R CNN
+F 0 "CR18" H 7700 4700 50  0000 R CNN
 F 1 "1SS352_H3FT" H 7900 4800 50  0000 R CNN
 F 2 "mypartsLib:1SS352_H3FT" H 7650 4700 60  0001 C CNN
@@
 AR Path="/5FD193EF/5FD2B5D0" Ref="CR27"  Part="1"
 AR Path="/5FD18D34/5FD2B5D0" Ref="CR17"  Part="1"
-F 0 "CR27" H 7700 4850 50  0000 R CNN
+F 0 "CR17" H 7700 4850 50  0000 R CNN
 F 1 "1SS352_H3FT" H 7900 4750 50  0000 R CNN
 F 2 "mypartsLib:1SS352_H3FT" H 7650 4350 60  0001 C CNN
@@
 AR Path="/5FD193EF/5FD0BC64" Ref="R91"  Part="1"
 AR Path="/5FD18D34/5FD0BC64" Ref="R65"  Part="1"
-F 0 "R91" V 8600 4550 50  0000 L CNN
+F 0 "R65" V 8600 4550 50  0000 L CNN
 F 1 "10k" V 8400 4550 50  0000 L CNN
 F 2 "Resistor_SMD:R_0603_1608Metric" V 8430 4600 50  0001 C CNN

Commit message: PCB Design Finished
Changed lines of the file:
@@
 $Descr A4 11693 8268
 encoding utf-8
-Sheet 6 17
+Sheet 9 17
 Title "rsp02_module_LoadSW_OCP_noOCP"
 Date "2020-12-07"
@@
 AR Path="/5FD193EF/5FD0BC5C" Ref="Q22"  Part="1"
 AR Path="/5FD18D34/5FD0BC5C" Ref="Q13"  Part="1"
-F 0 "Q13" H 7900 1617 50  0000 C CNN
+F 0 "Q22" H 7900 1617 50  0000 C CNN
 F 1 "SISS23DN-T1-GE3" H 7900 1526 50  0000 C CNN
 F 2 "mypartsLib:POWERPAK-1212-8" H 7900 800 50  0001 C CNN
@@
 AR Path="/5FD193EF/5FD0BC5D" Ref="R90"  Part="1"
 AR Path="/5FD18D34/5FD0BC5D" Ref="R64"  Part="1"
-F 0 "R64" H 7000 1750 50  0000 L CNN
+F 0 "R90" H 7000 1750 50  0000 L CNN
 F 1 "100k" H 7000 1550 50  0000 L CNN
 F 2 "Resistor_SMD:R_0603_1608Metric" V 6880 1650 50  0001 C CNN
@@
 AR Path="/5FD193EF/5FD0BC5E" Ref="R93"  Part="1"
 AR Path="/5FD18D34/5FD0BC5E" Ref="R67"  Part="1"
-F 0 "R67" H 9300 2250 50  0000 L CNN
+F 0 "R93" H 9300 2250 50  0000 L CNN
 F 1 "100k" H 9300 2050 50  0000 L CNN
 F 2 "Resistor_SMD:R_0603_1608Metric" V 9180 2150 50  0001 C CNN
@@
 AR Path="/5FD193EF/5FD0BC5F" Ref="R92"  Part="1"
 AR Path="/5FD18D34/5FD0BC5F" Ref="R66"  Part="1"
-F 0 "R66" H 8850 5000 50  0000 L CNN
+F 0 "R92" H 8850 5000 50  0000 L CNN
 F 1 "10k" H 8850 4800 50  0000 L CNN
 F 2 "Resistor_SMD:R_0603_1608Metric" V 8730 4900 50  0001 C CNN
@@
 AR Path="/5FD193EF/5FD2B5CE" Ref="Q24"  Part="1"
 AR Path="/5FD18D34/5FD2B5CE" Ref="Q15"  Part="1"
-F 0 "Q15" H 9294 4646 50  0000 L CNN
+F 0 "Q24" H 9294 4646 50  0000 L CNN
 F 1 "BC848B" H 9294 4555 50  0000 L CNN
 F 2 "Package_TO_SOT_SMD:SOT-23" H 8950 5100 50  0001 L CNN
@@
 AR Path="/5FD193EF/5FD2B5CD" Ref="Q23"  Part="1"
 AR Path="/5FD18D34/5FD2B5CD" Ref="Q14"  Part="1"
-F 0 "Q14" H 7705 2404 50  0000 L CNN
+F 0 "Q23" H 7705 2404 50  0000 L CNN
 F 1 "IRF7404" H 7705 2495 50  0000 L CNN
 F 2 "Package_SO:SOIC-8_3.9x4.9mm_P1.27mm" H 7700 2375 50  0001 L CIN
@@
 AR Path="/5FD193EF/5FD2B5CF" Ref="CR28"  Part="1"
 AR Path="/5FD18D34/5FD2B5CF" Ref="CR18"  Part="1"
-F 0 "CR18" H 7700 4700 50  0000 R CNN
+F 0 "CR28" H 7700 4700 50  0000 R CNN
 F 1 "1SS352_H3FT" H 7900 4800 50  0000 R CNN
 F 2 "mypartsLib:1SS352_H3FT" H 7650 4700 60  0001 C CNN
@@
 AR Path="/5FD193EF/5FD2B5D0" Ref="CR27"  Part="1"
 AR Path="/5FD18D34/5FD2B5D0" Ref="CR17"  Part="1"
-F 0 "CR17" H 7700 4850 50  0000 R CNN
+F 0 "CR27" H 7700 4850 50  0000 R CNN
 F 1 "1SS352_H3FT" H 7900 4750 50  0000 R CNN
 F 2 "mypartsLib:1SS352_H3FT" H 7650 4350 60  0001 C CNN
@@
 AR Path="/5FD193EF/5FD0BC64" Ref="R91"  Part="1"
 AR Path="/5FD18D34/5FD0BC64" Ref="R65"  Part="1"
-F 0 "R65" V 8600 4550 50  0000 L CNN
+F 0 "R91" V 8600 4550 50  0000 L CNN
 F 1 "10k" V 8400 4550 50  0000 L CNN
 F 2 "Resistor_SMD:R_0603_1608Metric" V 8430 4600 50  0001 C CNN
