File: rsp02_LoadSW_OCP_Circuit_v1_2.kicad_pcb (KiCad board)
At the start: 2 copper layers, 40 x 20 mm, 30 parts, among them IC1 OP291GSZ_v2, J1 Conn_01x02, J2 Conn_01x04, J3 Conn_01x02, J4 Conn_01x02, Q1 SISS23DN-T1-GE3, Q2 IRF7404, Q3 BC848B

Commit message: Update PCB
Parts:
- removed REF1, REF2, REF3, REF4: MountingHole_2.2mm_M2_ISO7380_Pad, MountingHole:MountingHole_2.2mm_M2_ISO7380_Pad
- added C10: 0.1u, Capacitor_SMD:C_0603_1608Metric, F.Cu at (222.1, 134.4)
- added C11: 0.1u, Capacitor_SMD:C_0603_1608Metric, F.Cu at (218.1, 136.9)
- added C12: 0.1u, Capacitor_SMD:C_0603_1608Metric, F.Cu at (222.1, 131.9)
- added C13: 0.1u, Capacitor_SMD:C_0603_1608Metric, F.Cu at (234.3, 87.8)
- added C14: 0.1u, Capacitor_SMD:C_0603_1608Metric, F.Cu at (238.3, 85.3)
- added C15: 0.1u, Capacitor_SMD:C_0603_1608Metric, F.Cu at (238.3, 87.8)
- added C16: 0.1u, Capacitor_SMD:C_0603_1608Metric, F.Cu at (174.8, 139.2)
- added C17: 0.1u, Capacitor_SMD:C_0603_1608Metric, F.Cu at (170.8, 139.2)
- added C18: 0.1u, Capacitor_SMD:C_0603_1608Metric, F.Cu at (180.2, 131.7)
- added C19: 0.1u, Capacitor_SMD:C_0603_1608Metric, F.Cu at (220.2, 149.7)
- added C20: 0.1u, Capacitor_SMD:C_0603_1608Metric, F.Cu at (233.5, 134.5)
- added C21: 0.1u, Capacitor_SMD:C_0603_1608Metric, F.Cu at (258.3, 106.6)
- added C22: 0.1u, Capacitor_SMD:C_0603_1608Metric, F.Cu at (208.1, 148.7)
- added C23: 0.1u, Capacitor_SMD:C_0603_1608Metric, F.Cu at (186.6, 149.7)
- added C24: 0.1u, Capacitor_SMD:C_0603_1608Metric, F.Cu at (151.6, 150.3)
- added C25: 0.1u, Capacitor_SMD:C_0603_1608Metric, F.Cu at (139.4, 149.3)
- added C26: 0.1u, Capacitor_SMD:C_0603_1608Metric, F.Cu at (165.7, 149.7)
- added C4: 0.1u, Capacitor_SMD:C_0603_1608Metric, F.Cu at (147.8, 127.4)
- added C5: 0.1u, Capacitor_SMD:C_0603_1608Metric, F.Cu at (152.9, 124.4)
- added C6: 0.1u, Capacitor_SMD:C_0603_1608Metric, F.Cu at (140.6, 135.4)
- added C7: 0.1u, Capacitor_SMD:C_0603_1608Metric, F.Cu at (242.3, 101.1)
- added C8: 0.1u, Capacitor_SMD:C_0603_1608Metric, F.Cu at (238.3, 108.2)
- added C9: 0.1u, Capacitor_SMD:C_0603_1608Metric, F.Cu at (230.3, 107.9)
- added CR10: 1SS352_H3FT, mypartsLib:1SS352_H3FT, F.Cu at (233.4, 95.9)
- added CR11: 1SS352_H3FT, mypartsLib:1SS352_H3FT, F.Cu at (216.3, 110.2)
- added CR12: 1SS352_H3FT, mypartsLib:1SS352_H3FT, F.Cu at (238.5, 95.9)
- added CR13: 1SS352_H3FT, mypartsLib:1SS352_H3FT, F.Cu at (222.3, 124.6)
- added CR14: 1SS352_H3FT, mypartsLib:1SS352_H3FT, F.Cu at (200.1, 138.9)
- added CR15: 1SS352_H3FT, mypartsLib:1SS352_H3FT, F.Cu at (217.3, 124.6)
- added CR16: 1SS352_H3FT, mypartsLib:1SS352_H3FT, F.Cu at (200.1, 136.0)
- added CR17: 1SS352_H3FT, mypartsLib:1SS352_H3FT, F.Cu at (250.2, 95.8)
- added CR18: 1SS352_H3FT, mypartsLib:1SS352_H3FT, F.Cu at (258.6, 89.3)
- added CR19: 1SS352_H3FT, mypartsLib:1SS352_H3FT, F.Cu at (233.4, 75.5)
- added CR20: 1SS352_H3FT, mypartsLib:1SS352_H3FT, F.Cu at (216.3, 86.8)
- added CR21: 1SS352_H3FT, mypartsLib:1SS352_H3FT, F.Cu at (216.3, 89.8)
- added CR22: 1SS352_H3FT, mypartsLib:1SS352_H3FT, F.Cu at (238.5, 75.5)
- added CR23: 1SS352_H3FT, mypartsLib:1SS352_H3FT, F.Cu at (166.2, 136.0)
- added CR24: 1SS352_H3FT, mypartsLib:1SS352_H3FT, F.Cu at (183.4, 124.6)
- added CR25: 1SS352_H3FT, mypartsLib:1SS352_H3FT, F.Cu at (166.2, 138.9)
- added CR26: 1SS352_H3FT, mypartsLib:1SS352_H3FT, F.Cu at (188.4, 124.6)
- added CR27: 1SS352_H3FT, mypartsLib:1SS352_H3FT, F.Cu at (234.0, 122.7)
- added CR28: 1SS352_H3FT, mypartsLib:1SS352_H3FT, F.Cu at (242.5, 116.3)
- added CR5: 1SS352_H3FT, mypartsLib:1SS352_H3FT, F.Cu at (131.2, 136.0)
- added CR6: 1SS352_H3FT, mypartsLib:1SS352_H3FT, F.Cu at (139.7, 131.1)
- added CR7: 1SS352_H3FT, mypartsLib:1SS352_H3FT, F.Cu at (131.2, 138.9)
- added CR8: 1SS352_H3FT, mypartsLib:1SS352_H3FT, F.Cu at (148.4, 124.6)
- added CR9: 1SS352_H3FT, mypartsLib:1SS352_H3FT, F.Cu at (216.3, 107.2)
- added IC10: INA199A1DCKT_v2, Package_TO_SOT_SMD:SOT-363_SC-70-6, F.Cu at (208.2, 145.5)
- added IC11: INA199A1DCKT_v2, Package_TO_SOT_SMD:SOT-363_SC-70-6, F.Cu at (191.4, 145.5)
- added IC12: INA199A1DCKT_v2, Package_TO_SOT_SMD:SOT-363_SC-70-6, F.Cu at (156.4, 146.1)
- added IC13: INA199A1DCKT_v2, Package_TO_SOT_SMD:SOT-363_SC-70-6, F.Cu at (139.5, 146.1)
- added IC14: INA199A1DCKT_v2, Package_TO_SOT_SMD:SOT-363_SC-70-6, F.Cu at (174.5, 145.5)
- added IC2: OP191GSZ_v2, Package_SO:SOIC-8_3.9x4.9mm_P1.27mm, F.Cu at (132.9, 131.3)
- added IC3: OP191GSZ_v2, Package_SO:SOIC-8_3.9x4.9mm_P1.27mm, F.Cu at (226.7, 97.6)
- added IC4: OP191GSZ_v2, Package_SO:SOIC-8_3.9x4.9mm_P1.27mm, F.Cu at (201.8, 131.3)
- added IC5: OP191GSZ_v2, Package_SO:SOIC-8_3.9x4.9mm_P1.27mm, F.Cu at (226.7, 77.2)
- added IC6: OP191GSZ_v2, Package_SO:SOIC-8_3.9x4.9mm_P1.27mm, F.Cu at (176.6, 126.4)
- added IC7: INA199A1DCKT_v2, Package_TO_SOT_SMD:SOT-363_SC-70-6, F.Cu at (225.0, 145.5)
- added IC8: INA199A1DCKT_v2, Package_TO_SOT_SMD:SOT-363_SC-70-6, F.Cu at (242.3, 130.3)
- added IC9: INA199A1DCKT_v2, Package_TO_SOT_SMD:SOT-363_SC-70-6, F.Cu at (258.5, 103.4)
- added J10: Conn_01x02, TerminalBlock_Phoenix:TerminalBlock_Phoenix_MKDS-3-2-5.08_1x02_P5.08mm_Horizontal, F.Cu at (274.5, 112.0)
- added J11: Conn_01x02, TerminalBlock_Phoenix:TerminalBlock_Phoenix_MKDS-3-2-5.08_1x02_P5.08mm_Horizontal, F.Cu at (274.8, 124.0)
- added J12: Conn_01x02, TerminalBlock_Phoenix:TerminalBlock_Phoenix_MKDS-3-2-5.08_1x02_P5.08mm_Horizontal, F.Cu at (275.5, 136.8)
- added J13: Conn_01x02, TerminalBlock_Phoenix:TerminalBlock_Phoenix_MKDS-3-2-5.08_1x02_P5.08mm_Horizontal, F.Cu at (275.0, 148.2)
- added J14: Conn_01x02, TerminalBlock_Phoenix:TerminalBlock_Phoenix_MKDS-3-2-5.08_1x02_P5.08mm_Horizontal, F.Cu at (275.0, 160.8)
- added J15: Conn_01x10, TerminalBlock_Phoenix:TerminalBlock_Phoenix_MKDS-3-10-5.08_1x10_P5.08mm_Horizontal, F.Cu at (199.5, 158.8)
- added J16: Conn_01x10, TerminalBlock_Phoenix:TerminalBlock_Phoenix_MKDS-3-10-5.08_1x10_P5.08mm_Horizontal, F.Cu at (146.0, 158.8)
- added J5: Conn_01x02, TerminalBlock_Phoenix:TerminalBlock_Phoenix_MKDS-3-2-5.08_1x02_P5.08mm_Horizontal, F.Cu at (180.0, 69.5)
- added J6: Conn_01x02, TerminalBlock_Phoenix:TerminalBlock_Phoenix_MKDS-3-2-5.08_1x02_P5.08mm_Horizontal, F.Cu at (192.2, 69.5)
- added J7: Conn_01x02, TerminalBlock_Phoenix:TerminalBlock_Phoenix_MKDS-3-2-5.08_1x02_P5.08mm_Horizontal, F.Cu at (274.5, 75.2)
- added J8: Conn_01x02, TerminalBlock_Phoenix:TerminalBlock_Phoenix_MKDS-3-2-5.08_1x02_P5.08mm_Horizontal, F.Cu at (274.2, 87.8)
- added J9: Conn_01x02, TerminalBlock_Phoenix:TerminalBlock_Phoenix_MKDS-3-2-5.08_1x02_P5.08mm_Horizontal, F.Cu at (274.2, 100.0)
- added Q10: SISS23DN-T1-GE3, mypartsLib:POWERPAK-1212-8, F.Cu at (217.2, 128.3)
- added Q11: IRF7404, Package_SO:SOIC-8_3.9x4.9mm_P1.27mm, F.Cu at (210.5, 126.4)
- added Q12: BC848B, Package_TO_SOT_SMD:SOT-23, F.Cu at (221.8, 128.4)
- added Q13: SISS23DN-T1-GE3, mypartsLib:POWERPAK-1212-8, F.Cu at (258.5, 93.0)
- added Q14: IRF7404, Package_SO:SOIC-8_3.9x4.9mm_P1.27mm, F.Cu at (251.9, 91.1)
- added Q15: BC848B, Package_TO_SOT_SMD:SOT-23, F.Cu at (263.4, 90.1)
- added Q16: SISS23DN-T1-GE3, mypartsLib:POWERPAK-1212-8, F.Cu at (233.3, 79.1)
- added Q17: IRF7404, Package_SO:SOIC-8_3.9x4.9mm_P1.27mm, F.Cu at (218.0, 82.1)
- added Q18: BC848B, Package_TO_SOT_SMD:SOT-23, F.Cu at (238.0, 79.2)
- added Q19: SISS23DN-T1-GE3, mypartsLib:POWERPAK-1212-8, F.Cu at (183.3, 128.3)
- added Q20: IRF7404, Package_SO:SOIC-8_3.9x4.9mm_P1.27mm, F.Cu at (167.9, 131.3)
- added Q21: BC848B, Package_TO_SOT_SMD:SOT-23, F.Cu at (187.9, 128.4)
- added Q22: SISS23DN-T1-GE3, mypartsLib:POWERPAK-1212-8, F.Cu at (242.4, 119.9)
- added Q23: IRF7404, Package_SO:SOIC-8_3.9x4.9mm_P1.27mm, F.Cu at (235.7, 118.0)
- added Q24: BC848B, Package_TO_SOT_SMD:SOT-23, F.Cu at (247.2, 117.1)
- added Q4: SISS23DN-T1-GE3, mypartsLib:POWERPAK-1212-8, F.Cu at (136.2, 136.7)
- added Q5: IRF7404, Package_SO:SOIC-8_3.9x4.9mm_P1.27mm, F.Cu at (141.6, 126.4)
- added Q6: BC848B, Package_TO_SOT_SMD:SOT-23, F.Cu at (144.4, 131.9)
- added Q7: SISS23DN-T1-GE3, mypartsLib:POWERPAK-1212-8, F.Cu at (233.3, 99.5)
- added Q8: IRF7404, Package_SO:SOIC-8_3.9x4.9mm_P1.27mm, F.Cu at (218.0, 102.5)
- added Q9: BC848B, Package_TO_SOT_SMD:SOT-23, F.Cu at (238.0, 99.6)
- added R10: 0, Resistor_SMD:R_0603_1608Metric, F.Cu at (142.7, 117.5)
- added R100: 0, Resistor_SMD:R_0603_1608Metric, F.Cu at (249.7, 107.6)
- added R101: 0, Resistor_SMD:R_0603_1608Metric, F.Cu at (253.7, 107.6)
- added R102: 0.02, Resistor_SMD:R_2512_6332Metric, F.Cu at (252.0, 103.9)
- added R103: 0, Resistor_SMD:R_0603_1608Metric, F.Cu at (203.4, 149.7)
- added R104: 0, Resistor_SMD:R_0603_1608Metric, F.Cu at (199.4, 149.7)
- added R105: 0.02, Resistor_SMD:R_2512_6332Metric, F.Cu at (201.7, 146.0)
- added R106: 0, Resistor_SMD:R_0603_1608Metric, F.Cu at (191.2, 148.7)
- added R107: 0, Resistor_SMD:R_0603_1608Metric, F.Cu at (182.5, 149.7)
- added R108: 0.02, Resistor_SMD:R_2512_6332Metric, F.Cu at (184.9, 146.0)
- added R109: 0, Resistor_SMD:R_0603_1608Metric, F.Cu at (156.2, 149.3)
- added R11: 0, Resistor_SMD:R_0603_1608Metric, F.Cu at (154.8, 115.0)
- added R110: 0, Resistor_SMD:R_0603_1608Metric, F.Cu at (147.5, 150.3)
- added R111: 0.02, Resistor_SMD:R_2512_6332Metric, F.Cu at (149.9, 146.6)
- added R112: 0, Resistor_SMD:R_0603_1608Metric, F.Cu at (130.7, 150.3)
- added R113: 0, Resistor_SMD:R_0603_1608Metric, F.Cu at (134.7, 150.3)
- added R114: 0.04, Resistor_SMD:R_2512_6332Metric, F.Cu at (133.0, 146.6)
- added R115: 0, Resistor_SMD:R_0603_1608Metric, F.Cu at (169.7, 149.7)
- added R116: 0, Resistor_SMD:R_0603_1608Metric, F.Cu at (174.4, 148.7)
- added R117: 0.02, Resistor_SMD:R_2512_6332Metric, F.Cu at (168.0, 146.0)
- added R12: 0, Resistor_SMD:R_0603_1608Metric, F.Cu at (150.8, 115.0)
- added R13: 0, Resistor_SMD:R_0603_1608Metric, F.Cu at (146.7, 115.0)
- added R14: 0, Resistor_SMD:R_0603_1608Metric, F.Cu at (142.7, 115.0)
- added R15: 0, Resistor_SMD:R_0603_1608Metric, F.Cu at (138.7, 115.0)
- added R16: 0, Resistor_SMD:R_0603_1608Metric, F.Cu at (134.7, 117.5)
- added R17: 0, Resistor_SMD:R_0603_1608Metric, F.Cu at (130.7, 117.5)
- added R18: 0, Resistor_SMD:R_0603_1608Metric, F.Cu at (134.7, 115.0)
- added R19: 0, Resistor_SMD:R_0603_1608Metric, F.Cu at (130.7, 115.0)
- added R20: 6k, Resistor_SMD:R_0603_1608Metric, F.Cu at (258.3, 75.3)
- added R21: 100k, Resistor_SMD:R_0603_1608Metric, F.Cu at (249.7, 80.1)
- added R22: 0.05, Resistor_SMD:R_2512_6332Metric, F.Cu at (252.0, 76.4)
- added R23: 50k, Resistor_SMD:R_0603_1608Metric, F.Cu at (249.7, 82.7)
- added R24: 1000k, Resistor_SMD:R_0603_1608Metric, F.Cu at (253.7, 80.1)
- added R25: 10k, Resistor_SMD:R_0603_1608Metric, F.Cu at (258.3, 77.8)
- added R26: 1k, Resistor_SMD:R_0603_1608Metric, F.Cu at (262.4, 75.3)
- added R27: 100k, Resistor_SMD:R_0603_1608Metric, F.Cu at (253.7, 82.7)
- added R28: 10k, Resistor_SMD:R_0603_1608Metric, F.Cu at (257.7, 80.3)
- added R29: 10k, Resistor_SMD:R_0603_1608Metric, F.Cu at (262.4, 77.8)
- added R30: 100k, Resistor_SMD:R_0603_1608Metric, F.Cu at (257.7, 82.8)
- added R31: 6k, Resistor_SMD:R_0603_1608Metric, F.Cu at (148.7, 134.9)
- added R32: 100k, Resistor_SMD:R_0603_1608Metric, F.Cu at (152.7, 129.9)
- added R33: 0.05, Resistor_SMD:R_2512_6332Metric, F.Cu at (133.0, 125.6)
- added R34: 50k, Resistor_SMD:R_0603_1608Metric, F.Cu at (155.9, 126.9)
- added R35: 1000k, Resistor_SMD:R_0603_1608Metric, F.Cu at (144.6, 137.9)
- added R36: 10k, Resistor_SMD:R_0603_1608Metric, F.Cu at (148.7, 129.9)
- added R37: 1k, Resistor_SMD:R_0603_1608Metric, F.Cu at (151.9, 127.4)
- added R38: 100k, Resistor_SMD:R_0603_1608Metric, F.Cu at (156.9, 124.4)
- added R39: 10k, Resistor_SMD:R_0603_1608Metric, F.Cu at (148.7, 132.4)
- added R40: 10k, Resistor_SMD:R_0603_1608Metric, F.Cu at (144.6, 135.4)
- added R41: 100k, Resistor_SMD:R_0603_1608Metric, F.Cu at (152.7, 132.4)
- added R42: 6k, Resistor_SMD:R_0603_1608Metric, F.Cu at (230.3, 102.9)
- added R43: 100k, Resistor_SMD:R_0603_1608Metric, F.Cu at (224.8, 110.4)
- added R44: 0.05, Resistor_SMD:R_2512_6332Metric, F.Cu at (218.1, 96.8)
- added R45: 50k, Resistor_SMD:R_0603_1608Metric, F.Cu at (220.8, 110.4)
- added R46: 1000k, Resistor_SMD:R_0603_1608Metric, F.Cu at (230.3, 105.4)
- added R47: 10k, Resistor_SMD:R_0603_1608Metric, F.Cu at (242.2, 98.6)
- added R48: 1k, Resistor_SMD:R_0603_1608Metric, F.Cu at (234.3, 105.7)
- added R49: 100k, Resistor_SMD:R_0603_1608Metric, F.Cu at (238.3, 105.7)
- added R50: 10k, Resistor_SMD:R_0603_1608Metric, F.Cu at (238.3, 103.2)
- added R51: 10k, Resistor_SMD:R_0603_1608Metric, F.Cu at (234.3, 103.2)
- added R52: 100k, Resistor_SMD:R_0603_1608Metric, F.Cu at (230.3, 110.4)
- added R53: 6k, Resistor_SMD:R_0603_1608Metric, F.Cu at (214.1, 139.2)
- added R54: 100k, Resistor_SMD:R_0603_1608Metric, F.Cu at (218.1, 131.9)
- added R55: 0.05, Resistor_SMD:R_2512_6332Metric, F.Cu at (201.9, 125.6)
- added R56: 50k, Resistor_SMD:R_0603_1608Metric, F.Cu at (208.7, 139.2)
- added R57: 1000k, Resistor_SMD:R_0603_1608Metric, F.Cu at (222.1, 136.9)
- added R58: 10k, Resistor_SMD:R_0603_1608Metric, F.Cu at (214.1, 131.7)
- added R59: 1k, Resistor_SMD:R_0603_1608Metric, F.Cu at (214.1, 134.2)
- added R60: 100k, Resistor_SMD:R_0603_1608Metric, F.Cu at (214.1, 136.7)
- added R61: 10k, Resistor_SMD:R_0603_1608Metric, F.Cu at (218.1, 134.4)
- added R62: 10k, Resistor_SMD:R_0603_1608Metric, F.Cu at (226.1, 127.4)
- added R63: 100k, Resistor_SMD:R_0603_1608Metric, F.Cu at (226.1, 129.9)
- added R64: 100k, Resistor_SMD:R_0603_1608Metric, F.Cu at (254.7, 96.4)
- added R65: 10k, Resistor_SMD:R_0603_1608Metric, F.Cu at (263.0, 93.7)
- added R66: 10k, Resistor_SMD:R_0603_1608Metric, F.Cu at (258.7, 96.4)
- added R67: 100k, Resistor_SMD:R_0603_1608Metric, F.Cu at (263.0, 96.2)
- added R68: 5.3k, Resistor_SMD:R_0603_1608Metric, F.Cu at (242.3, 80.7)
- added R69: 100k, Resistor_SMD:R_0603_1608Metric, F.Cu at (230.3, 90.0)
- added R70: 0.10, Resistor_SMD:R_2512_6332Metric, F.Cu at (218.1, 76.4)
- added R71: 50k, Resistor_SMD:R_0603_1608Metric, F.Cu at (220.8, 90.1)
- added R72: 1000k, Resistor_SMD:R_0603_1608Metric, F.Cu at (224.8, 90.1)
- added R73: 10k, Resistor_SMD:R_0603_1608Metric, F.Cu at (230.3, 82.5)
- added R74: 1k, Resistor_SMD:R_0603_1608Metric, F.Cu at (230.3, 85.0)
- added R75: 100k, Resistor_SMD:R_0603_1608Metric, F.Cu at (230.3, 87.5)
- added R76: 10k, Resistor_SMD:R_0603_1608Metric, F.Cu at (234.3, 82.8)
- added R77: 10k, Resistor_SMD:R_0603_1608Metric, F.Cu at (234.3, 85.3)
- added R78: 100k, Resistor_SMD:R_0603_1608Metric, F.Cu at (242.2, 78.2)
- added R79: 6k, Resistor_SMD:R_0603_1608Metric, F.Cu at (180.2, 139.2)
- added R80: 100k, Resistor_SMD:R_0603_1608Metric, F.Cu at (180.2, 134.2)
- added R81: 0.05, Resistor_SMD:R_2512_6332Metric, F.Cu at (168.0, 125.6)
- added R82: 50k, Resistor_SMD:R_0603_1608Metric, F.Cu at (180.2, 136.7)
- added R83: 1000k, Resistor_SMD:R_0603_1608Metric, F.Cu at (184.2, 134.4)
- added R84: 10k, Resistor_SMD:R_0603_1608Metric, F.Cu at (192.2, 127.4)
- added R85: 1k, Resistor_SMD:R_0603_1608Metric, F.Cu at (188.2, 131.9)
- added R86: 100k, Resistor_SMD:R_0603_1608Metric, F.Cu at (184.2, 136.9)
- added R87: 10k, Resistor_SMD:R_0603_1608Metric, F.Cu at (188.2, 134.4)
- added R88: 10k, Resistor_SMD:R_0603_1608Metric, F.Cu at (192.2, 129.9)
- added R89: 100k, Resistor_SMD:R_0603_1608Metric, F.Cu at (188.2, 136.9)
- added R9: 0, Resistor_SMD:R_0603_1608Metric, F.Cu at (138.7, 117.5)
- added R90: 100k, Resistor_SMD:R_0603_1608Metric, F.Cu at (246.8, 123.1)
- added R91: 10k, Resistor_SMD:R_0603_1608Metric, F.Cu at (242.6, 123.3)
- added R92: 10k, Resistor_SMD:R_0603_1608Metric, F.Cu at (246.8, 120.6)
- added R93: 100k, Resistor_SMD:R_0603_1608Metric, F.Cu at (238.6, 123.3)
- added R94: 0, Resistor_SMD:R_0603_1608Metric, F.Cu at (224.9, 148.7)
- added R95: 0, Resistor_SMD:R_0603_1608Metric, F.Cu at (216.2, 149.7)
- added R96: 0.02, Resistor_SMD:R_2512_6332Metric, F.Cu at (218.6, 146.0)
- added R97: 0, Resistor_SMD:R_0603_1608Metric, F.Cu at (237.5, 134.5)
- added R98: 0, Resistor_SMD:R_0603_1608Metric, F.Cu at (242.2, 133.5)
- added R99: 0.02, Resistor_SMD:R_2512_6332Metric, F.Cu at (235.8, 130.8)
- added RV3: 200k, Potentiometer_SMD:Potentiometer_Bourns_3314G_Vertical, F.Cu at (225.2, 105.0)
- added RV4: 200k, Potentiometer_SMD:Potentiometer_Bourns_3314G_Vertical, F.Cu at (209.1, 133.8)
- added RV5: 200k, Potentiometer_SMD:Potentiometer_Bourns_3314G_Vertical, F.Cu at (225.2, 84.6)
- added RV6: 200k, Potentiometer_SMD:Potentiometer_Bourns_3314G_Vertical, F.Cu at (175.2, 133.8)
- added Rh2: 100k, Resistor_SMD:R_0603_1608Metric, F.Cu at (140.6, 137.9)
- added Rh3: 100k, Resistor_SMD:R_0603_1608Metric, F.Cu at (234.3, 108.2)
- added Rh4: 100k, Resistor_SMD:R_0603_1608Metric, F.Cu at (204.7, 139.2)
- added Rh5: 100k, Resistor_SMD:R_0603_1608Metric, F.Cu at (238.3, 82.8)
- added Rh6: 100k, Resistor_SMD:R_0603_1608Metric, F.Cu at (184.2, 131.9)
- C1, C2, C3: footprint Capacitor_SMD:C_0402_1005Metric -> Capacitor_SMD:C_0603_1608Metric
- IC1: value OP291GSZ_v2 -> OP191GSZ_v2
- J1, J3, J4: footprint Connector_PinHeader_2.00mm:PinHeader_1x02_P2.00mm_Vertical -> TerminalBlock_Phoenix:TerminalBlock_Phoenix_MKDS-3-2-5.08_1x02_P5.08mm_Horizontal
- J2: value Conn_01x04 -> Conn_01x02; footprint Connector_PinHeader_2.00mm:PinHeader_1x04_P2.00mm_Vertical -> TerminalBlock_Phoenix:TerminalBlock_Phoenix_MKDS-3-2-5.08_1x02_P5.08mm_Horizontal
- R1, R6, R8: value 100k -> 0; footprint Resistor_SMD:R_0402_1005Metric -> Resistor_SMD:R_0603_1608Metric
- R2: value 0.5 -> 0; footprint Resistor_SMD:R_2512_6332Metric -> Resistor_SMD:R_0603_1608Metric
- R3: value 1000k -> 0; footprint Resistor_SMD:R_0402_1005Metric -> Resistor_SMD:R_0603_1608Metric
- R4, R7: value 10k -> 0; footprint Resistor_SMD:R_0402_1005Metric -> Resistor_SMD:R_0603_1608Metric
- R5: value 1k -> 0; footprint Resistor_SMD:R_0402_1005Metric -> Resistor_SMD:R_0603_1608Metric
- RV1, RV2: value 100k -> 200k
- Rh1: footprint Resistor_SMD:R_0402_1005Metric -> Resistor_SMD:R_0603_1608Metric
- moved J3 50.6 mm to (118.8, 127.0), turned to 270 degrees
- moved J2 41.1 mm to (118.8, 114.6), turned to 270 degrees
- moved R3 32.2 mm to (170.9, 109.1)
- moved R6 29.9 mm to (174.9, 109.1)
- moved R1 29.3 mm to (166.9, 109.1), turned to 0 degrees
- moved R2 29.2 mm to (166.9, 111.6), turned to 0 degrees
- moved RV2 29.1 mm to (167.9, 100.4)
- moved R5 27.1 mm to (170.9, 111.6)
- moved J4 26.4 mm to (168.2, 69.5), turned to 180 degrees
- moved R4 22.6 mm to (166.9, 114.1), turned to 0 degrees
- moved R8 22.5 mm to (174.9, 111.6)
- moved CR1 21.5 mm to (150.9, 97.7), turned to 0 degrees
- moved Q2 19.9 mm to (138.1, 105.9)
- moved J1 19.6 mm to (118.8, 101.8), turned to 270 degrees
- moved R7 19.5 mm to (170.9, 114.1), turned to 0 degrees
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Connections:
- C2 pad 1: Vinput -> /Power_Line_3_3V_RX
- C3 pad 1: Voutput -> Power_RX
- CR3 pad 2: IOexpander -> /LoadSW_OCP_RX/LSWE1
- CR4 pad 2: ReceiverRx -> /LoadSW_OCP_RX/LSWE2
- IC1 pad 1: Net-(CR2-Pad2) -> Net-(IC1-Pad1)
- IC1 pad 6: Net-(IC1-Pad6) -> Net-(CR2-Pad2)
- IC1 pad 7: Net-(IC1-Pad7) -> /Power_Line_3_3V_RX
- IC1 pad 8: Vinput -> Net-(IC1-Pad8)
- J1 pad 1: Vinput -> GNDA
- J1 pad 2: GNDA -> Power_IN_5_0V
- J2 pad 1: Voutput -> GNDA
- J2 pad 2: Net-(J2-Pad2) -> Power_IN_3_3V
- J3 pad 1: IOexpander -> GNDA
- J3 pad 2: GNDA -> Power_IN_3_0V
- J4 pad 1: ReceiverRx -> Power_Mon_5_0V
- Q1 pad 5: Voutput -> Power_RX
- Q1 pad 6: Voutput -> Power_RX
- Q1 pad 7: Voutput -> Power_RX
- Q1 pad 8: Voutput -> Power_RX
- Q3 pad 1: Net-(CR3-Pad1) -> Net-(Q3-Pad1)
- R1 pad 1: Net-(IC1-Pad3) -> Power_IN_5_0V
- R1 pad 2: GNDA -> Power_Mon_5_0V
- R2 pad 1: Net-(CR1-Pad1) -> Power_IN_3_3V
- R2 pad 2: Vinput -> Power_Mon_3_3V
- R3 pad 1: Net-(C1-Pad1) -> Power_IN_3_0V
- R3 pad 2: GNDA -> Power_Mon_3_0V
- R4 pad 1: Net-(C3-Pad2) -> /LoadSW_OCP_TX PA/LSWE1
- R4 pad 2: Net-(CR2-Pad2) -> TPASWE_fromIOE
- R5 pad 1: Net-(CR2-Pad1) -> /LoadSW_OCP_TX PA/LSWE2
- R5 pad 2: Net-(C3-Pad2) -> /Power_Line_5_0V_TXPA
- R6 pad 1: Net-(CR1-Pad1) -> /LoadSW_OCP_TX/LSWE1
- R6 pad 2: Net-(Q1-Pad4) -> TXSWE_fromIOE
- R7 pad 1: Net-(CR3-Pad1) -> /LoadSW_OCP_TX/LSWE2
- R7 pad 2: GNDA -> TXSWE_fromRX
- R8 pad 1: Vinput -> /LoadSW_OCP_RX/LSWE1
- R8 pad 2: Net-(Q2-Pad4) -> /Power_Line_3_3V_RX
- RV1 pad 1: Vinput -> Net-(CR1-Pad1)
- RV1 pad 2: Vinput -> Net-(CR1-Pad1)
- RV1 pad 3: Net-(IC1-Pad3) -> Net-(R23-Pad1)
- RV2 pad 1: Net-(CR1-Pad1) -> Net-(CR5-Pad1)
- RV2 pad 2: Net-(CR1-Pad1) -> Net-(CR5-Pad1)
- RV2 pad 3: Net-(C1-Pad1) -> Net-(R34-Pad1)
Routing:
- net Net-(CR1-Pad1): track 48.3 -> 0.00 mm, vias 3 -> 0
- net Vinput: track 45.4 -> 0.00 mm, vias 3 -> 0
- net Net-(CR2-Pad1): track 43.7 -> 0.00 mm, vias 4 -> 0
- net Net-(IC1-Pad3): track 24.8 -> 0.00 mm, vias 3 -> 0
- net Net-(Q1-Pad4): track 22.1 -> 0.00 mm, vias 2 -> 0
- net Net-(CR2-Pad2): track 21.7 -> 0.00 mm, vias 2 -> 0
- net Net-(C1-Pad1): track 20.9 -> 0.00 mm
- net Net-(CR3-Pad1): track 16.8 -> 0.00 mm
- net Voutput: track 16.4 -> 0.00 mm
- net Net-(Q2-Pad4): track 11.7 -> 0.00 mm
- net IOexpander: track 10.4 -> 0.00 mm
- net ReceiverRx: track 8.80 -> 0.00 mm
- net Net-(C3-Pad2): track 7.47 -> 0.00 mm
- net GNDA: track 4.21 -> 0.00 mm, vias 24 -> 0
- removed copper zone on B.Cu, net GNDA
- removed copper zone on F.Cu, net GNDA
Other:
- board outline removed

Commit message: PCB Update
Parts:
- J4, J5, J6: footprint TerminalBlock_Phoenix:TerminalBlock_Phoenix_MKDS-3-2-5.08_1x02_P5.08mm_Horizontal -> Connector_PinHeader_2.54mm:PinHeader_1x02_P2.54mm_Vertical
- moved CR18 182.9 mm to (138.5, 227.3)
- moved CR17 182.9 mm to (130.1, 233.8)
- moved Q14 182.9 mm to (131.8, 229.1)
- moved R64 182.9 mm to (134.6, 234.3)
- moved R66 182.9 mm to (138.6, 234.3)
- moved R67 182.9 mm to (142.9, 234.1)
- moved Q15 182.9 mm to (143.3, 228.1)
- moved R65 182.9 mm to (142.9, 231.6)
- moved Q13 178.7 mm to (135.3, 222.5)
- moved IC9 176.6 mm to (99.5, 180.5), turned to 180 degrees
- moved C21 171.9 mm to (102.8, 179.9), turned to 270 degrees
- moved J15 170.8 mm to (161.0, -7.62), turned to 180 degrees
- moved R100 167.8 mm to (96.6, 176.5), turned to 90 degrees
- moved R102 166.8 mm to (99.7, 172.0)
- moved R101 166.0 mm to (102.6, 176.4), turned to 90 degrees
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Connections:
- net Net-(CR1-Pad1) renamed /LoadSW_OCP_RX/Power_Line
- net Net-(CR13-Pad1) renamed /LoadSW_OCP_Attitude/Power_Line
- net Net-(CR19-Pad1) renamed /LoadSW_OCP_TX PA/Power_Line
- net Net-(CR23-Pad1) renamed /LoadSW_OCP_TX/Power_Line
- net Net-(CR5-Pad1) renamed /LoadSW_OCP_Mission OBC/Power_Line
- net Net-(CR9-Pad1) renamed /LoadSW_OCP_C&DH OBC/Power_Line
- J1 pad 1: GNDA -> Power_IN_5_0V
- J1 pad 2: Power_IN_5_0V -> GNDA
- J2 pad 1: GNDA -> Power_IN_3_3V
- J2 pad 2: Power_IN_3_3V -> GNDA
- J3 pad 1: GNDA -> Power_IN_3_0V
- J3 pad 2: Power_IN_3_0V -> GNDA
Routing:
- net /LoadSW_OCP_TX PA/Power_Line: track 0.00 -> 57.6 mm
- net Power_TX_PA: track 0.00 -> 48.1 mm
- net Power_IN_5_0V: track 0.00 -> 25.0 mm
- net /Power_Line_5_0V_TXPA: track 0.00 -> 13.4 mm
- net Net-(CR21-Pad1): track 0.00 -> 7.43 mm
- net Net-(Q18-Pad1): track 0.00 -> 6.43 mm
- net Net-(C13-Pad1): track 0.00 -> 5.53 mm
- net Net-(IC13-Pad5): track 0.00 -> 5.47 mm
- net Net-(IC13-Pad4): track 0.00 -> 3.17 mm
- net Net-(R71-Pad1): track 0.00 -> 2.88 mm
- net Net-(IC5-Pad3): track 0.00 -> 2.41 mm
- net Net-(Q17-Pad4): track 0.00 -> 2.22 mm
- net /LoadSW_OCP_TX PA/LSWE1: track 0.00 -> 2.13 mm
- net /LoadSW_OCP_TX PA/LSWE2: track 0.00 -> 2.05 mm
- net (no net): track 0.00 -> 2.04 mm

Commit message: PCB Update
Parts:
- J15: footprint TerminalBlock_Phoenix:TerminalBlock_Phoenix_MKDS-3-10-5.08_1x10_P5.08mm_Horizontal -> Connector_PinHeader_2.54mm:PinHeader_1x10_P2.54mm_Vertical
- moved J15 146.4 mm to (66.8, 104.4)
- moved J16 106.4 mm to (68.5, 147.8), turned to 270 degrees
- moved J6 92.0 mm to (66.8, 75.4)
- moved J5 82.3 mm to (66.8, 66.8)
- moved CR26 73.2 mm to (83.5, 81.5), turned to 180 degrees
- moved J4 72.6 mm to (66.8, 58.1)
- moved R88 70.7 mm to (87.9, 81.7), turned to 270 degrees
- moved CR4 70.6 mm to (83.2, 109.1), turned to 180 degrees
- moved CR3 64.4 mm to (83.3, 104.9), turned to 180 degrees
- moved R87 63.3 mm to (88.6, 77.3), turned to 180 degrees
- moved R29 62.4 mm to (87.9, 108.9), turned to 270 degrees
- moved Q21 61.9 mm to (92.8, 79.6)
- moved CR12 59.5 mm to (83.3, 163.3), turned to 180 degrees
- moved R89 56.7 mm to (96.1, 81.6), turned to 90 degrees
- moved R20 56.6 mm to (88.5, 94.2), turned to 270 degrees
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Connections:
- IC12 pad 6: Imon_TX -> Imon_RX
- J15 pad 8: Imon_TX -> Imon_RX
Routing:
- net Power_IN_3_3V: track 0.00 -> 209.3 mm
- net TXSWE_fromRX: track 0.00 -> 189.0 mm, vias 0 -> 2
- net TPASWE_fromIOE: track 0.00 -> 155.9 mm, vias 0 -> 1
- net Imon_NicWire: track 0.00 -> 143.5 mm, vias 0 -> 2
- net Power_Mon_3_0V: track 0.00 -> 132.5 mm, vias 0 -> 2
- net Imon_DplyCvr: track 0.00 -> 126.1 mm, vias 0 -> 4
- net TXSWE_fromIOE: track 0.00 -> 121.8 mm, vias 0 -> 1
- net Imon_Attde: track 0.00 -> 101.8 mm, vias 0 -> 2
- net NWSWE_fromRX: track 0.00 -> 88.3 mm, vias 0 -> 2
- net Power_NichromeWire: track 0.00 -> 80.2 mm
- net /Power_Line_3_3V_RX: track 0.00 -> 79.0 mm, vias 0 -> 5
- net /Power_Line_3_3V_M: track 0.00 -> 78.4 mm, vias 0 -> 6
- net /Power_Line_3_3V_C: track 0.00 -> 76.6 mm, vias 0 -> 5
- net NWSWE_fromIOE: track 0.00 -> 75.0 mm, vias 0 -> 1
- net Imon_CDH: track 0.00 -> 74.0 mm, vias 0 -> 4
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Other:
- board text added: "3.0V INPUT"
- board text added: "3.0V Input Monitor"
- board text added: "3.0V OUT DplyCvr"
- board text added: "3.0V OUT NicWire"
- board text added: "3.3V INPUT"
- board text added: "3.3V Input Monitor"
- board text added: "3.3V OUT Attitude"
- board text added: "3.3V OUT C&DH"
- board text added: "3.3V OUT Misson"
- board text added: "3.3V OUT RX"
- board text added: "3.3V OUT TX"
- board text added: "5.0V INPUT"
- board text added: "5.0V Input Monitor"
- board text added: "5.0V OUT TXPA"
- board text added: "Control from IOExpander/RX"
- board text added: "Current Sense Monitor"

Commit message: PCB Design Finished
Parts:
- added G***: LOGO, mypartsLib:rsp_logo_small, F.Cu at (71.5, 221.7)
- added REF1: MountingHole_2.2mm_M2_ISO7380_Pad, MountingHole:MountingHole_2.2mm_M2_ISO7380_Pad, F.Cu at (62.9, 32.9)
- added REF2: MountingHole_2.2mm_M2_ISO7380_Pad, MountingHole:MountingHole_2.2mm_M2_ISO7380_Pad, F.Cu at (124.0, 47.0)
- added REF3: MountingHole_2.2mm_M2_ISO7380_Pad, MountingHole:MountingHole_2.2mm_M2_ISO7380_Pad, F.Cu at (124.0, 226.0)
- added REF4: MountingHole_2.2mm_M2_ISO7380_Pad, MountingHole:MountingHole_2.2mm_M2_ISO7380_Pad, F.Cu at (62.6, 225.1)
Connections:
- R11 pad 2: /Power_Line_3_3V_M -> Net-(R11-Pad2)
- R15 pad 2: /Power_Line_3_3V_A -> Net-(R15-Pad2)
- R17 pad 2: /Power_Line_3_0V_DplyCvr -> Net-(R17-Pad2)
- R5 pad 2: /Power_Line_5_0V_TXPA -> Net-(R5-Pad2)
Routing:
- net /Power_Line_3_3V_M: track 78.4 -> 55.4 mm, vias 6 -> 3
- net /Power_Line_3_3V_A: track 72.9 -> 52.3 mm, vias 4 -> 3
- net /Power_Line_5_0V_TXPA: track 68.9 -> 51.3 mm, vias 5 -> 3
- net /Power_Line_3_0V_DplyCvr: track 73.6 -> 62.8 mm
- net Power_TX: track 37.4 -> 45.0 mm
- net Power_NichromeWire: track 80.2 -> 80.9 mm
- net Imon_NicWire: track 143.5 -> 144.2 mm
- net GNDA: vias 0 -> 190
- added copper zone on B.Cu, net GNDA
- added copper zone on F.Cu, net GNDA
Other:
- board outline added: 70 x 200 mm

Commit message: before gerber output
Routing:
- net Power_Attitude: track 47.0 -> 76.8 mm
- net Power_RX: track 41.7 -> 69.4 mm
- net Power_C&DH: track 42.7 -> 69.9 mm
- net Power_Mission: track 46.4 -> 72.3 mm
- net Power_TX: track 45.0 -> 68.8 mm
- net Power_TX_PA: track 48.1 -> 68.8 mm
- net /LoadSW_OCP_TX PA/Power_Line: track 65.2 -> 77.9 mm
- net /LoadSW_OCP_RX/Power_Line: track 62.9 -> 75.0 mm
- net /LoadSW_OCP_TX/Power_Line: track 61.9 -> 73.3 mm
- net /LoadSW_OCP_Mission OBC/Power_Line: track 58.8 -> 68.8 mm
- net /LoadSW_OCP_C&DH OBC/Power_Line: track 55.8 -> 65.9 mm
- net /Power_Line_3_3V_TX: track 57.3 -> 66.5 mm
- net /Power_Line_3_3V_RX: track 79.0 -> 88.2 mm
- net /Power_Line_3_3V_C: track 76.6 -> 85.8 mm
- net /Power_Line_3_3V_M: track 55.4 -> 64.2 mm
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
Commit message: PCB reUpdate
Parts:
- added R118: 1k, Resistor_SMD:R_0603_1608Metric, F.Cu at (86.5, 92.6)
- added R119: 1k, Resistor_SMD:R_0603_1608Metric, F.Cu at (86.3, 120.0)
- added R120: 1k, Resistor_SMD:R_0603_1608Metric, F.Cu at (86.5, 147.0)
- added R121: 1k, Resistor_SMD:R_0603_1608Metric, F.Cu at (87.7, 172.6)
- added R122: 300, Resistor_SMD:R_0603_1608Metric, F.Cu at (87.4, 38.8)
- added R123: 1k, Resistor_SMD:R_0603_1608Metric, F.Cu at (87.3, 66.7)
- R20, R31, R42, R53, R79: value 6k -> 5k
- R68: value 5.3k -> 5k
- moved R53 2.30 mm to (88.4, 177.0)
- moved R42 1.73 mm to (88.5, 149.6)
- moved R43 1.52 mm to (88.5, 153.1)
- moved R54 1.48 mm to (88.4, 180.8)
- moved R31 1.28 mm to (88.7, 122.4)
- moved R20 1.23 mm to (88.9, 95.4)
- moved R32 1.03 mm to (88.7, 126.2)
- moved R21 0.84 mm to (88.9, 99.1)
- moved R68 0.61 mm to (89.1, 41.5)
Connections:
- R20 pad 1: /Power_Line_3_3V_RX -> Net-(R118-Pad2)
- R31 pad 1: /Power_Line_3_3V_M -> Net-(R119-Pad2)
- R42 pad 1: /Power_Line_3_3V_C -> Net-(R120-Pad2)
- R53 pad 1: /Power_Line_3_3V_A -> Net-(R121-Pad2)
- R68 pad 1: /Power_Line_5_0V_TXPA -> Net-(R122-Pad2)
- R79 pad 1: /Power_Line_3_3V_TX -> Net-(R123-Pad2)
Routing:
- net Net-(R121-Pad2): track 0.00 -> 3.63 mm
- net Net-(R118-Pad2): track 0.00 -> 3.17 mm
- net /Power_Line_3_3V_TX: track 66.5 -> 69.7 mm
- net Net-(R119-Pad2): track 0.00 -> 2.86 mm
- net /Power_Line_3_3V_A: track 58.7 -> 61.5 mm
- net Net-(R120-Pad2): track 0.00 -> 2.77 mm
- net Net-(R122-Pad2): track 0.00 -> 2.63 mm
- net Net-(R123-Pad2): track 0.00 -> 2.46 mm
- net /Power_Line_5_0V_TXPA: track 58.6 -> 61.0 mm
- net Net-(IC4-Pad3): track 26.6 -> 25.0 mm
- net Net-(IC3-Pad3): track 27.5 -> 26.1 mm
- net /Power_Line_3_3V_RX: track 88.2 -> 89.4 mm
- net /Power_Line_3_3V_M: track 64.2 -> 63.3 mm
- net /Power_Line_3_3V_C: track 85.8 -> 86.6 mm
- net Net-(IC5-Pad3): track 26.7 -> 26.1 mm
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