File: rsp02_module_LoadSW_OCP_3_3V.sch (KiCad schematic (older format))
At the start: 23 parts, among them IC1 OP291GSZ_v2, Q1 SISS23DN-T1-GE3, Q2 IRF7404, Q3 BC848B

Commit message: Update
Parts:
- removed C2, C3: 0.1u, Capacitor_SMD:C_0402_1005Metric, symbol Device:C
- removed R2: 0.5, Resistor_SMD:R_2512_6332Metric, symbol Device:R
- removed R3: 1000k, Resistor_SMD:R_0402_1005Metric, symbol Device:R
- removed R4: 10k, Resistor_SMD:R_0402_1005Metric, symbol Device:R
- removed R5: 1k, Resistor_SMD:R_0402_1005Metric, symbol Device:R
- removed RV2: 100k, Potentiometer_SMD:Potentiometer_Bourns_3314G_Vertical, symbol Device:R_Potentiometer_Trim
- removed Rh1: 100k, Resistor_SMD:R_0402_1005Metric, symbol Device:R
- added C20, C21: 0.1u, Capacitor_SMD:C_0402_1005Metric, symbol Device:C
- added R75: 0.5, Resistor_SMD:R_2512_6332Metric, symbol Device:R
- added R76: 1000k, Resistor_SMD:R_0402_1005Metric, symbol Device:R
- added R77: 10k, Resistor_SMD:R_0402_1005Metric, symbol Device:R
- added R78: 1k, Resistor_SMD:R_0402_1005Metric, symbol Device:R
- added RV14: 100k, Potentiometer_SMD:Potentiometer_Bourns_3314G_Vertical, symbol Device:R_Potentiometer_Trim
- added Rh7: 100k, Resistor_SMD:R_0402_1005Metric, symbol Device:R
- renumbered C1 to C19, CR1 to CR25, CR2 to CR26, CR3 to CR27, CR4 to CR28, IC1 to IC7, Q1 to Q19, Q2 to Q20, Q3 to Q21, R1 to R74, R6 to R79, R9 to R80, R7 to R81, R8 to R82, RV1 to RV13
Connections:
- net GND: now also C20.2, R76.2
- net INPUT: now also C20.1, R75.2
- net OUTPUT: now also C21.1
- net at C19.1, CR25.2 (anode), IC7.2 (-INA): now also R76.1, RV14.3
- net at CR25.1 (cathode), Q19.1 (S(1)), Q19.2 (S(2))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: now also R75.1, RV14.1, RV14.2
- net at CR26.1 (cathode), Q20.5 (D), Q20.6 (D)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: now also R78.1
- net at CR26.2 (anode), IC7.1 (OUTA): now also R77.2, Rh7.1
- net at IC7.3 (+INA), R74.1, RV13.3: now also Rh7.2
- new net: C21.2, R77.1, R78.2

Commit message: Update Design
Parts:
- removed CR27, CR28: 1SS352_H3FT, mypartsLib:1SS352_H3FT, symbol mypartsLib:1SS352_H3FT
- removed IC7: OP291GSZ_v2, Package_SO:SOIC-8_3.9x4.9mm_P1.27mm, symbol mypartsLib:OP291GSZ_v2
- removed RV13: 100k, Potentiometer_SMD:Potentiometer_Bourns_3314G_Vertical, symbol Device:R_Potentiometer_Trim
- added CR25, CR26: 1SS352_H3FT, mypartsLib:1SS352_H3FT, symbol mypartsLib:1SS352_H3FT
- added IC6: OP191GSZ_v2, SOIC127P600X175-8N, symbol mypartsLib:OP191GSZ_v2
- added R79: 6k, Resistor_SMD:R_0402_1005Metric, symbol Device:R
- added R82: 50k, Resistor_SMD:R_0402_1005Metric, symbol Device:R
- R81: renamed from R75; value 0.5 -> 0.05
- RV6: renamed from RV14; value 100k -> 200k
- renumbered C19 to C16, C20 to C17, C21 to C18, CR25 to CR23, CR26 to CR24, R74 to R80, R76 to R83, R77 to R84, R78 to R85, R79 to R86, R80 to R87, R81 to R88, R82 to R89, Rh7 to Rh6
Connections:
- net GND: now also IC6.4 (-V)
- net INPUT: now also IC6.7 (+V), R79.1
- net LSWE1: now also CR25.2 (anode)
- net LSWE2: now also CR26.2 (anode)
- net at C16.1, CR23.2 (anode), R83.1: now also IC6.2 (-INA), R82.2; no longer RV6.3
- net at CR24.2 (anode), R84.2, Rh6.1: now also IC6.6 (OUTA)
- net at R80.1, Rh6.2: now also IC6.3 (+INA), R79.2
- net at R87.2: now also CR25.1 (cathode), CR26.1 (cathode)
- new net: R82.1, RV6.3
- no-connect marks 3 -> 0
Other:
- moved on the sheet: C17, RV6

Commit message: Update PCB
Parts:
- C16, C17, C18: footprint Capacitor_SMD:C_0402_1005Metric -> Capacitor_SMD:C_0603_1608Metric
- IC6: footprint SOIC127P600X175-8N -> Package_SO:SOIC-8_3.9x4.9mm_P1.27mm
- R79, R80, R82, R83, R84, R85, R86, R87, R88, R89, Rh6: footprint Resistor_SMD:R_0402_1005Metric -> Resistor_SMD:R_0603_1608Metric
Changed lines of the file:
@@
 $Descr A4 11693 8268
 encoding utf-8
-Sheet 2 17
+Sheet 3 17
 Title "rsp02_module_LoadSW_OCP_3_3V"
 Date "2020-12-06"
@@
 AR Path="/5FD1935C/60873804" Ref="R35"  Part="1"
 AR Path="/5FD19389/60873804" Ref="R46"  Part="1"
-F 0 "R83" H 3550 4950 50  0000 L CNN
+F 0 "R35" H 3550 4950 50  0000 L CNN
 F 1 "1000k" H 3550 4750 50  0000 L CNN
-F 2 "Resistor_SMD:R_0402_1005Metric" V 3430 4850 50  0001 C CNN
+F 2 "Resistor_SMD:R_0603_1608Metric" V 3430 4850 50  0001 C CNN
 F 3 "~" H 3500 4850 50  0001 C CNN
 	1    3500 4850
@@
 AR Path="/5FD1935C/60873805" Ref="C5"  Part="1"
 AR Path="/5FD19389/60873805" Ref="C8"  Part="1"
-F 0 "C17" H 4950 5350 50  0000 L CNN
+F 0 "C5" H 4950 5350 50  0000 L CNN
 F 1 "0.1u" H 4950 5150 50  0000 L CNN
-F 2 "Capacitor_SMD:C_0402_1005Metric" H 4888 5100 50  0001 C CNN
+F 2 "Capacitor_SMD:C_0603_1608Metric" H 4888 5100 50  0001 C CNN
 F 3 "~" H 4850 5250 50  0001 C CNN
 	1    4850 5250
@@
 AR Path="/5FD1935C/60873806" Ref="R33"  Part="1"
 AR Path="/5FD19389/60873806" Ref="R44"  Part="1"
-F 0 "R81" V 2800 1270 50  0000 L CNN
+F 0 "R33" V 2800 1270 50  0000 L CNN
 F 1 "0.05" V 3000 1260 50  0000 L CNN
 F 2 "Resistor_SMD:R_2512_6332Metric" V 2830 1350 50  0001 C CNN
@@
 AR Path="/5FD1935C/60873807" Ref="R37"  Part="1"
 AR Path="/5FD19389/60873807" Ref="R48"  Part="1"
-F 0 "R85" H 6700 3050 50  0000 L CNN
+F 0 "R37" H 6700 3050 50  0000 L CNN
 F 1 "1k" H 6700 2850 50  0000 L CNN
-F 2 "Resistor_SMD:R_0402_1005Metric" V 6580 2950 50  0001 C CNN
+F 2 "Resistor_SMD:R_0603_1608Metric" V 6580 2950 50  0001 C CNN
 F 3 "~" H 6650 2950 50  0001 C CNN
 	1    6650 2950
@@
 AR Path="/5FD1935C/60873808" Ref="Rh2"  Part="1"
 AR Path="/5FD19389/60873808" Ref="Rh3"  Part="1"
-F 0 "Rh6" V 4500 2100 50  0000 L CNN
+F 0 "Rh2" V 4500 2100 50  0000 L CNN
 F 1 "100k" V 4700 2050 50  0000 L CNN
-F 2 "Resistor_SMD:R_0402_1005Metric" V 4530 2150 50  0001 C CNN
+F 2 "Resistor_SMD:R_0603_1608Metric" V 4530 2150 50  0001 C CNN
 F 3 "~" H 4600 2150 50  0001 C CNN
 	1    4600 2150
@@
 AR Path="/5FD1935C/60873809" Ref="C6"  Part="1"
 AR Path="/5FD19389/60873809" Ref="C9"  Part="1"
-F 0 "C18" V 7500 3750 50  0000 L CNN
+F 0 "C6" V 7500 3750 50  0000 L CNN
 F 1 "0.1u" V 7800 3750 50  0000 L CNN
-F 2 "Capacitor_SMD:C_0402_1005Metric" H 7688 3650 50  0001 C CNN
+F 2 "Capacitor_SMD:C_0603_1608Metric" H 7688 3650 50  0001 C CNN
 F 3 "~" H 7650 3800 50  0001 C CNN
 	1    7650 3800
@@
 AR Path="/5FD1935C/6087380A" Ref="R36"  Part="1"
 AR Path="/5FD19389/6087380A" Ref="R47"  Part="1"
-F 0 "R84" V 6150 3750 50  0000 L CNN
+F 0 "R36" V 6150 3750 50  0000 L CNN
 F 1 "10k" V 6350 3750 50  0000 L CNN
-F 2 "Resistor_SMD:R_0402_1005Metric" V 6180 3800 50  0001 C CNN
+F 2 "Resistor_SMD:R_0603_1608Metric" V 6180 3800 50  0001 C CNN
 F 3 "~" H 6250 3800 50  0001 C CNN
 	1    6250 3800
@@
 AR Path="/5FD1935C/5FD2B5C2" Ref="R32"  Part="1"
 AR Path="/5FD19389/5FD2B5C2" Ref="R43"  Part="1"
-F 0 "R80" H 2350 4950 50  0000 L CNN
+F 0 "R32" H 2350 4950 50  0000 L CNN
 F 1 "100k" H 2350 4750 50  0000 L CNN
-F 2 "Resistor_SMD:R_0402_1005Metric" V 2230 4850 50  0001 C CNN
+F 2 "Resistor_SMD:R_0603_1608Metric" V 2230 4850 50  0001 C CNN
 F 3 "~" H 2300 4850 50  0001 C CNN
 	1    2300 4850
@@
 AR Path="/5FD1935C/5F5E905F" Ref="C4"  Part="1"
 AR Path="/5FD19389/5F5E905F" Ref="C7"  Part="1"
-F 0 "C16" H 4000 4950 50  0000 L CNN
+F 0 "C4" H 4000 4950 50  0000 L CNN
 F 1 "0.1u" H 4000 4750 50  0000 L CNN
-F 2 "Capacitor_SMD:C_0402_1005Metric" H 3938 4700 50  0001 C CNN
+F 2 "Capacitor_SMD:C_0603_1608Metric" H 3938 4700 50  0001 C CNN
 F 3 "~" H 3900 4850 50  0001 C CNN
 	1    3900 4850
@@
 AR Path="/5FD1935C/5F64B0A6" Ref="Q4"  Part="1"
 AR Path="/5FD19389/5F64B0A6" Ref="Q7"  Part="1"
-F 0 "Q19" H 7900 1617 50  0000 C CNN
+F 0 "Q4" H 7900 1617 50  0000 C CNN
 F 1 "SISS23DN-T1-GE3" H 7900 1526 50  0000 C CNN
 F 2 "mypartsLib:POWERPAK-1212-8" H 7900 800 50  0001 C CNN
@@
 AR Path="/5FD1935C/5F671DB4" Ref="R38"  Part="1"
 AR Path="/5FD19389/5F671DB4" Ref="R49"  Part="1"
-F 0 "R86" H 7000 1750 50  0000 L CNN
+F 0 "R38" H 7000 1750 50  0000 L CNN
 F 1 "100k" H 7000 1550 50  0000 L CNN
-F 2 "Resistor_SMD:R_0402_1005Metric" V 6880 1650 50  0001 C CNN
+F 2 "Resistor_SMD:R_0603_1608Metric" V 6880 1650 50  0001 C CNN
 F 3 "~" H 6950 1650 50  0001 C CNN
 	1    6950 1650
@@
 AR Path="/5FD1935C/5F67CD1A" Ref="R41"  Part="1"
 AR Path="/5FD19389/5F67CD1A" Ref="R52"  Part="1"
-F 0 "R89" H 9300 2250 50  0000 L CNN
+F 0 "R41" H 9300 2250 50  0000 L CNN
 F 1 "100k" H 9300 2050 50  0000 L CNN
-F 2 "Resistor_SMD:R_0402_1005Metric" V 9180 2150 50  0001 C CNN
+F 2 "Resistor_SMD:R_0603_1608Metric" V 9180 2150 50  0001 C CNN
 F 3 "~" H 9250 2150 50  0001 C CNN
 	1    9250 2150
@@
 AR Path="/5FD1935C/5F6AFC79" Ref="R40"  Part="1"
 AR Path="/5FD19389/5F6AFC79" Ref="R51"  Part="1"
-F 0 "R88" H 8850 5000 50  0000 L CNN
+F 0 "R40" H 8850 5000 50  0000 L CNN
 F 1 "10k" H 8850 4800 50  0000 L CNN
-F 2 "Resistor_SMD:R_0402_1005Metric" V 8730 4900 50  0001 C CNN
+F 2 "Resistor_SMD:R_0603_1608Metric" V 8730 4900 50  0001 C CNN
 F 3 "~" H 8800 4900 50  0001 C CNN
 	1    8800 4900
@@
 AR Path="/5FD1935C/60873814" Ref="RV2"  Part="1"
 AR Path="/5FD19389/60873814" Ref="RV3"  Part="1"
-F 0 "RV6" H 3431 2846 50  0000 R CNN
+F 0 "RV2" H 3431 2846 50  0000 R CNN
 F 1 "200k" H 3431 2755 50  0000 R CNN
 F 2 "Potentiometer_SMD:Potentiometer_Bourns_3314G_Vertical" H 3500 2800 50  0001 C CNN
@@
 AR Path="/5FD1935C/5FD0BC61" Ref="Q6"  Part="1"
 AR Path="/5FD19389/5FD0BC61" Ref="Q9"  Part="1"
-F 0 "Q21" H 9294 4646 50  0000 L CNN
+F 0 "Q6" H 9294 4646 50  0000 L CNN
 F 1 "BC848B" H 9294 4555 50  0000 L CNN
 F 2 "Package_TO_SOT_SMD:SOT-23" H 8950 5100 50  0001 L CNN
@@
 AR Path="/5FD1935C/5FD2B5C8" Ref="CR6"  Part="1"
 AR Path="/5FD19389/5FD2B5C8" Ref="CR10"  Part="1"
-F 0 "CR24" V 6356 2046 50  0000 R CNN
+F 0 "CR6" V 6356 2046 50  0000 R CNN
 F 1 "1SS352_H3FT" V 6250 2046 50  0000 R CNN
 F 2 "mypartsLib:1SS352_H3FT" H 6250 1900 60  0001 C CNN
@@
 AR Path="/5FD1935C/5FD2B5C9" Ref="CR5"  Part="1"
 AR Path="/5FD19389/5FD2B5C9" Ref="CR9"  Part="1"
-F 0 "CR23" V 4356 3096 50  0000 R CNN
+F 0 "CR5" V 4356 3096 50  0000 R CNN
 F 1 "1SS352_H3FT" V 4250 3096 50  0000 R CNN
 F 2 "mypartsLib:1SS352_H3FT" H 4250 2950 60  0001 C CNN
@@
 AR Path="/5FD1935C/5FD0BC60" Ref="Q5"  Part="1"
 AR Path="/5FD19389/5FD0BC60" Ref="Q8"  Part="1"
-F 0 "Q20" H 7705 2404 50  0000 L CNN
+F 0 "Q5" H 7705 2404 50  0000 L CNN
 F 1 "IRF7404" H 7705 2495 50  0000 L CNN
 F 2 "Package_SO:SOIC-8_3.9x4.9mm_P1.27mm" H 7700 2375 50  0001 L CIN
@@
 AR Path="/5FD1935C/5FD0BC62" Ref="CR8"  Part="1"
 AR Path="/5FD19389/5FD0BC62" Ref="CR12"  Part="1"
-F 0 "CR26" H 7700 4700 50  0000 R CNN
+F 0 "CR8" H 7700 4700 50  0000 R CNN
 F 1 "1SS352_H3FT" H 7900 4800 50  0000 R CNN
 F 2 "mypartsLib:1SS352_H3FT" H 7650 4700 60  0001 C CNN
@@
 AR Path="/5FD1935C/5FD0BC63" Ref="CR7"  Part="1"
 AR Path="/5FD19389/5FD0BC63" Ref="CR11"  Part="1"
-F 0 "CR25" H 7700 4850 50  0000 R CNN
+F 0 "CR7" H 7700 4850 50  0000 R CNN
 F 1 "1SS352_H3FT" H 7900 4750 50  0000 R CNN
 F 2 "mypartsLib:1SS352_H3FT" H 7650 4350 60  0001 C CNN
@@
 AR Path="/5FD1935C/5FD2B5D1" Ref="R39"  Part="1"
 AR Path="/5FD19389/5FD2B5D1" Ref="R50"  Part="1"
-F 0 "R87" V 8600 4550 50  0000 L CNN
+F 0 "R39" V 8600 4550 50  0000 L CNN
 F 1 "10k" V 8400 4550 50  0000 L CNN
-F 2 "Resistor_SMD:R_0402_1005Metric" V 8430 4600 50  0001 C CNN
+F 2 "Resistor_SMD:R_0603_1608Metric" V 8430 4600 50  0001 C CNN
 F 3 "~" H 8500 4600 50  0001 C CNN
 	1    8500 4600
@@
 AR Path="/5FD19389/5FD1BC90" Ref="IC3"  Part="1"
 AR Path="/5FD193BD/5FD1BC90" Ref="IC4"  Part="1"
-F 0 "IC6" H 5150 4865 50  0000 C CNN
+F 0 "IC2" H 5150 4865 50  0000 C CNN
 F 1 "OP191GSZ_v2" H 5150 4774 50  0000 C CNN
-F 2 "SOIC127P600X175-8N" H 5750 4650 50  0001 L CNN
+F 2 "Package_SO:SOIC-8_3.9x4.9mm_P1.27mm" H 5750 4650 50  0001 L CNN
 F 3 "http://uk.rs-online.com/web/p/products/0427284P" H 5700 4350 50  0001 L CNN
 F 4 "Analog Devices OP191GSZ Op Amp, 3MHz Rail-Rail, 3  9 V, 8-Pin SOIC" H 5750 4450 50  0001 L CNN "Description"
@@
 AR Path="/5FD1935C/5FD3743B" Ref="R31"  Part="1"
 AR Path="/5FD19389/5FD3743B" Ref="R42"  Part="1"
-F 0 "R79" H 2350 3100 50  0000 L CNN
+F 0 "R31" H 2350 3100 50  0000 L CNN
 F 1 "6k" H 2350 2900 50  0000 L CNN
-F 2 "Resistor_SMD:R_0402_1005Metric" V 2230 3000 50  0001 C CNN
+F 2 "Resistor_SMD:R_0603_1608Metric" V 2230 3000 50  0001 C CNN
 F 3 "~" H 2300 3000 50  0001 C CNN
 	1    2300 3000
@@
 AR Path="/5FD1935C/5FD25536" Ref="R34"  Part="1"
 AR Path="/5FD19389/5FD25536" Ref="R45"  Part="1"
-F 0 "R82" H 3550 3250 50  0000 L CNN
+F 0 "R34" H 3550 3250 50  0000 L CNN
 F 1 "50k" H 3550 3050 50  0000 L CNN
-F 2 "Resistor_SMD:R_0402_1005Metric" V 3430 3150 50  0001 C CNN
+F 2 "Resistor_SMD:R_0603_1608Metric" V 3430 3150 50  0001 C CNN
 F 3 "~" H 3500 3150 50  0001 C CNN
 	1    3500 3150

Commit message: PCB Update
Connections:
- net Power_Line: now reaches CR23.1 (cathode), Q19.1 (S(1)), Q19.2 (S(2)), Q19.3 (S(3)), R81.1, R86.1, RV6.1, RV6.2
Changed lines of the file:
@@
 $Descr A4 11693 8268
 encoding utf-8
-Sheet 3 17
+Sheet 8 17
 Title "rsp02_module_LoadSW_OCP_3_3V"
 Date "2020-12-06"
@@
 AR Path="/5FD1935C/60873804" Ref="R35"  Part="1"
 AR Path="/5FD19389/60873804" Ref="R46"  Part="1"
-F 0 "R35" H 3550 4950 50  0000 L CNN
+F 0 "R83" H 3550 4950 50  0000 L CNN
 F 1 "1000k" H 3550 4750 50  0000 L CNN
 F 2 "Resistor_SMD:R_0603_1608Metric" V 3430 4850 50  0001 C CNN
@@
 AR Path="/5FD1935C/60873805" Ref="C5"  Part="1"
 AR Path="/5FD19389/60873805" Ref="C8"  Part="1"
-F 0 "C5" H 4950 5350 50  0000 L CNN
+F 0 "C17" H 4950 5350 50  0000 L CNN
 F 1 "0.1u" H 4950 5150 50  0000 L CNN
 F 2 "Capacitor_SMD:C_0603_1608Metric" H 4888 5100 50  0001 C CNN
@@
 AR Path="/5FD1935C/60873806" Ref="R33"  Part="1"
 AR Path="/5FD19389/60873806" Ref="R44"  Part="1"
-F 0 "R33" V 2800 1270 50  0000 L CNN
+F 0 "R81" V 2800 1270 50  0000 L CNN
 F 1 "0.05" V 3000 1260 50  0000 L CNN
 F 2 "Resistor_SMD:R_2512_6332Metric" V 2830 1350 50  0001 C CNN
@@
 AR Path="/5FD1935C/60873807" Ref="R37"  Part="1"
 AR Path="/5FD19389/60873807" Ref="R48"  Part="1"
-F 0 "R37" H 6700 3050 50  0000 L CNN
+F 0 "R85" H 6700 3050 50  0000 L CNN
 F 1 "1k" H 6700 2850 50  0000 L CNN
 F 2 "Resistor_SMD:R_0603_1608Metric" V 6580 2950 50  0001 C CNN
@@
 AR Path="/5FD1935C/60873808" Ref="Rh2"  Part="1"
 AR Path="/5FD19389/60873808" Ref="Rh3"  Part="1"
-F 0 "Rh2" V 4500 2100 50  0000 L CNN
+F 0 "Rh6" V 4500 2100 50  0000 L CNN
 F 1 "100k" V 4700 2050 50  0000 L CNN
 F 2 "Resistor_SMD:R_0603_1608Metric" V 4530 2150 50  0001 C CNN
@@
 AR Path="/5FD1935C/60873809" Ref="C6"  Part="1"
 AR Path="/5FD19389/60873809" Ref="C9"  Part="1"
-F 0 "C6" V 7500 3750 50  0000 L CNN
+F 0 "C18" V 7500 3750 50  0000 L CNN
 F 1 "0.1u" V 7800 3750 50  0000 L CNN
 F 2 "Capacitor_SMD:C_0603_1608Metric" H 7688 3650 50  0001 C CNN
@@
 AR Path="/5FD1935C/6087380A" Ref="R36"  Part="1"
 AR Path="/5FD19389/6087380A" Ref="R47"  Part="1"
-F 0 "R36" V 6150 3750 50  0000 L CNN
+F 0 "R84" V 6150 3750 50  0000 L CNN
 F 1 "10k" V 6350 3750 50  0000 L CNN
 F 2 "Resistor_SMD:R_0603_1608Metric" V 6180 3800 50  0001 C CNN
@@
 AR Path="/5FD1935C/5FD2B5C2" Ref="R32"  Part="1"
 AR Path="/5FD19389/5FD2B5C2" Ref="R43"  Part="1"
-F 0 "R32" H 2350 4950 50  0000 L CNN
+F 0 "R80" H 2350 4950 50  0000 L CNN
 F 1 "100k" H 2350 4750 50  0000 L CNN
 F 2 "Resistor_SMD:R_0603_1608Metric" V 2230 4850 50  0001 C CNN
@@
 AR Path="/5FD1935C/5F5E905F" Ref="C4"  Part="1"
 AR Path="/5FD19389/5F5E905F" Ref="C7"  Part="1"
-F 0 "C4" H 4000 4950 50  0000 L CNN
+F 0 "C16" H 4000 4950 50  0000 L CNN
 F 1 "0.1u" H 4000 4750 50  0000 L CNN
 F 2 "Capacitor_SMD:C_0603_1608Metric" H 3938 4700 50  0001 C CNN
@@
 AR Path="/5FD1935C/5F64B0A6" Ref="Q4"  Part="1"
 AR Path="/5FD19389/5F64B0A6" Ref="Q7"  Part="1"
-F 0 "Q4" H 7900 1617 50  0000 C CNN
+F 0 "Q19" H 7900 1617 50  0000 C CNN
 F 1 "SISS23DN-T1-GE3" H 7900 1526 50  0000 C CNN
 F 2 "mypartsLib:POWERPAK-1212-8" H 7900 800 50  0001 C CNN
@@
 AR Path="/5FD1935C/5F671DB4" Ref="R38"  Part="1"
 AR Path="/5FD19389/5F671DB4" Ref="R49"  Part="1"
-F 0 "R38" H 7000 1750 50  0000 L CNN
+F 0 "R86" H 7000 1750 50  0000 L CNN
 F 1 "100k" H 7000 1550 50  0000 L CNN
 F 2 "Resistor_SMD:R_0603_1608Metric" V 6880 1650 50  0001 C CNN
@@
 AR Path="/5FD1935C/5F67CD1A" Ref="R41"  Part="1"
 AR Path="/5FD19389/5F67CD1A" Ref="R52"  Part="1"
-F 0 "R41" H 9300 2250 50  0000 L CNN
+F 0 "R89" H 9300 2250 50  0000 L CNN
 F 1 "100k" H 9300 2050 50  0000 L CNN
 F 2 "Resistor_SMD:R_0603_1608Metric" V 9180 2150 50  0001 C CNN
@@
 AR Path="/5FD1935C/5F6AFC79" Ref="R40"  Part="1"
 AR Path="/5FD19389/5F6AFC79" Ref="R51"  Part="1"
-F 0 "R40" H 8850 5000 50  0000 L CNN
+F 0 "R88" H 8850 5000 50  0000 L CNN
 F 1 "10k" H 8850 4800 50  0000 L CNN
 F 2 "Resistor_SMD:R_0603_1608Metric" V 8730 4900 50  0001 C CNN
@@
 AR Path="/5FD1935C/60873814" Ref="RV2"  Part="1"
 AR Path="/5FD19389/60873814" Ref="RV3"  Part="1"
-F 0 "RV2" H 3431 2846 50  0000 R CNN
+F 0 "RV6" H 3431 2846 50  0000 R CNN
 F 1 "200k" H 3431 2755 50  0000 R CNN
 F 2 "Potentiometer_SMD:Potentiometer_Bourns_3314G_Vertical" H 3500 2800 50  0001 C CNN
@@
 AR Path="/5FD1935C/5FD0BC61" Ref="Q6"  Part="1"
 AR Path="/5FD19389/5FD0BC61" Ref="Q9"  Part="1"
-F 0 "Q6" H 9294 4646 50  0000 L CNN
+F 0 "Q21" H 9294 4646 50  0000 L CNN
 F 1 "BC848B" H 9294 4555 50  0000 L CNN
 F 2 "Package_TO_SOT_SMD:SOT-23" H 8950 5100 50  0001 L CNN
@@
 AR Path="/5FD1935C/5FD2B5C8" Ref="CR6"  Part="1"
 AR Path="/5FD19389/5FD2B5C8" Ref="CR10"  Part="1"
-F 0 "CR6" V 6356 2046 50  0000 R CNN
+F 0 "CR24" V 6356 2046 50  0000 R CNN
 F 1 "1SS352_H3FT" V 6250 2046 50  0000 R CNN
 F 2 "mypartsLib:1SS352_H3FT" H 6250 1900 60  0001 C CNN
@@
 AR Path="/5FD1935C/5FD2B5C9" Ref="CR5"  Part="1"
 AR Path="/5FD19389/5FD2B5C9" Ref="CR9"  Part="1"
-F 0 "CR5" V 4356 3096 50  0000 R CNN
+F 0 "CR23" V 4356 3096 50  0000 R CNN
 F 1 "1SS352_H3FT" V 4250 3096 50  0000 R CNN
 F 2 "mypartsLib:1SS352_H3FT" H 4250 2950 60  0001 C CNN
@@
 AR Path="/5FD1935C/5FD0BC60" Ref="Q5"  Part="1"
 AR Path="/5FD19389/5FD0BC60" Ref="Q8"  Part="1"
-F 0 "Q5" H 7705 2404 50  0000 L CNN
+F 0 "Q20" H 7705 2404 50  0000 L CNN
 F 1 "IRF7404" H 7705 2495 50  0000 L CNN
 F 2 "Package_SO:SOIC-8_3.9x4.9mm_P1.27mm" H 7700 2375 50  0001 L CIN
@@
 AR Path="/5FD1935C/5FD0BC62" Ref="CR8"  Part="1"
 AR Path="/5FD19389/5FD0BC62" Ref="CR12"  Part="1"
-F 0 "CR8" H 7700 4700 50  0000 R CNN
+F 0 "CR26" H 7700 4700 50  0000 R CNN
 F 1 "1SS352_H3FT" H 7900 4800 50  0000 R CNN
 F 2 "mypartsLib:1SS352_H3FT" H 7650 4700 60  0001 C CNN
@@
 AR Path="/5FD1935C/5FD0BC63" Ref="CR7"  Part="1"
 AR Path="/5FD19389/5FD0BC63" Ref="CR11"  Part="1"
-F 0 "CR7" H 7700 4850 50  0000 R CNN
+F 0 "CR25" H 7700 4850 50  0000 R CNN
 F 1 "1SS352_H3FT" H 7900 4750 50  0000 R CNN
 F 2 "mypartsLib:1SS352_H3FT" H 7650 4350 60  0001 C CNN
@@
 AR Path="/5FD1935C/5FD2B5D1" Ref="R39"  Part="1"
 AR Path="/5FD19389/5FD2B5D1" Ref="R50"  Part="1"
-F 0 "R39" V 8600 4550 50  0000 L CNN
+F 0 "R87" V 8600 4550 50  0000 L CNN
 F 1 "10k" V 8400 4550 50  0000 L CNN
 F 2 "Resistor_SMD:R_0603_1608Metric" V 8430 4600 50  0001 C CNN
@@
 AR Path="/5FD19389/5FD1BC90" Ref="IC3"  Part="1"
 AR Path="/5FD193BD/5FD1BC90" Ref="IC4"  Part="1"
-F 0 "IC2" H 5150 4865 50  0000 C CNN
+F 0 "IC6" H 5150 4865 50  0000 C CNN
 F 1 "OP191GSZ_v2" H 5150 4774 50  0000 C CNN
 F 2 "Package_SO:SOIC-8_3.9x4.9mm_P1.27mm" H 5750 4650 50  0001 L CNN
@@
 AR Path="/5FD1935C/5FD3743B" Ref="R31"  Part="1"
 AR Path="/5FD19389/5FD3743B" Ref="R42"  Part="1"
-F 0 "R31" H 2350 3100 50  0000 L CNN
+F 0 "R79" H 2350 3100 50  0000 L CNN
 F 1 "6k" H 2350 2900 50  0000 L CNN
 F 2 "Resistor_SMD:R_0603_1608Metric" V 2230 3000 50  0001 C CNN
@@
 AR Path="/5FD1935C/5FD25536" Ref="R34"  Part="1"
 AR Path="/5FD19389/5FD25536" Ref="R45"  Part="1"
-F 0 "R34" H 3550 3250 50  0000 L CNN
+F 0 "R82" H 3550 3250 50  0000 L CNN
 F 1 "50k" H 3550 3050 50  0000 L CNN
 F 2 "Resistor_SMD:R_0603_1608Metric" V 3430 3150 50  0001 C CNN
@@
 Wire Wire Line
 	3500 3000 3500 2950
+Text Label 4580 1350 0    50   ~ 0
+Power_Line
 $EndSCHEMATC
