File: rsp02_module_LoadSW_OCP_3_3V.sch (KiCad schematic (older format))
At the start: 24 parts, among them IC6 OP191GSZ_v2, Q19 SISS23DN-T1-GE3, Q20 IRF7404, Q21 BC848B

Commit message: PCB Update
Changed lines of the file:
@@
 $Descr A4 11693 8268
 encoding utf-8
-Sheet 8 17
+Sheet 2 17
 Title "rsp02_module_LoadSW_OCP_3_3V"
 Date "2020-12-06"
@@
 AR Path="/5FD1935C/60873804" Ref="R35"  Part="1"
 AR Path="/5FD19389/60873804" Ref="R46"  Part="1"
-F 0 "R83" H 3550 4950 50  0000 L CNN
+F 0 "R24" H 3550 4950 50  0000 L CNN
 F 1 "1000k" H 3550 4750 50  0000 L CNN
 F 2 "Resistor_SMD:R_0603_1608Metric" V 3430 4850 50  0001 C CNN
@@
 AR Path="/5FD1935C/60873805" Ref="C5"  Part="1"
 AR Path="/5FD19389/60873805" Ref="C8"  Part="1"
-F 0 "C17" H 4950 5350 50  0000 L CNN
+F 0 "C2" H 4950 5350 50  0000 L CNN
 F 1 "0.1u" H 4950 5150 50  0000 L CNN
 F 2 "Capacitor_SMD:C_0603_1608Metric" H 4888 5100 50  0001 C CNN
@@
 AR Path="/5FD1935C/60873806" Ref="R33"  Part="1"
 AR Path="/5FD19389/60873806" Ref="R44"  Part="1"
-F 0 "R81" V 2800 1270 50  0000 L CNN
+F 0 "R22" V 2800 1270 50  0000 L CNN
 F 1 "0.05" V 3000 1260 50  0000 L CNN
 F 2 "Resistor_SMD:R_2512_6332Metric" V 2830 1350 50  0001 C CNN
@@
 AR Path="/5FD1935C/60873807" Ref="R37"  Part="1"
 AR Path="/5FD19389/60873807" Ref="R48"  Part="1"
-F 0 "R85" H 6700 3050 50  0000 L CNN
+F 0 "R26" H 6700 3050 50  0000 L CNN
 F 1 "1k" H 6700 2850 50  0000 L CNN
 F 2 "Resistor_SMD:R_0603_1608Metric" V 6580 2950 50  0001 C CNN
@@
 AR Path="/5FD1935C/60873808" Ref="Rh2"  Part="1"
 AR Path="/5FD19389/60873808" Ref="Rh3"  Part="1"
-F 0 "Rh6" V 4500 2100 50  0000 L CNN
+F 0 "Rh1" V 4500 2100 50  0000 L CNN
 F 1 "100k" V 4700 2050 50  0000 L CNN
 F 2 "Resistor_SMD:R_0603_1608Metric" V 4530 2150 50  0001 C CNN
@@
 AR Path="/5FD1935C/60873809" Ref="C6"  Part="1"
 AR Path="/5FD19389/60873809" Ref="C9"  Part="1"
-F 0 "C18" V 7500 3750 50  0000 L CNN
+F 0 "C3" V 7500 3750 50  0000 L CNN
 F 1 "0.1u" V 7800 3750 50  0000 L CNN
 F 2 "Capacitor_SMD:C_0603_1608Metric" H 7688 3650 50  0001 C CNN
@@
 AR Path="/5FD1935C/6087380A" Ref="R36"  Part="1"
 AR Path="/5FD19389/6087380A" Ref="R47"  Part="1"
-F 0 "R84" V 6150 3750 50  0000 L CNN
+F 0 "R25" V 6150 3750 50  0000 L CNN
 F 1 "10k" V 6350 3750 50  0000 L CNN
 F 2 "Resistor_SMD:R_0603_1608Metric" V 6180 3800 50  0001 C CNN
@@
 AR Path="/5FD1935C/5FD2B5C2" Ref="R32"  Part="1"
 AR Path="/5FD19389/5FD2B5C2" Ref="R43"  Part="1"
-F 0 "R80" H 2350 4950 50  0000 L CNN
+F 0 "R21" H 2350 4950 50  0000 L CNN
 F 1 "100k" H 2350 4750 50  0000 L CNN
 F 2 "Resistor_SMD:R_0603_1608Metric" V 2230 4850 50  0001 C CNN
@@
 AR Path="/5FD1935C/5F5E905F" Ref="C4"  Part="1"
 AR Path="/5FD19389/5F5E905F" Ref="C7"  Part="1"
-F 0 "C16" H 4000 4950 50  0000 L CNN
+F 0 "C1" H 4000 4950 50  0000 L CNN
 F 1 "0.1u" H 4000 4750 50  0000 L CNN
 F 2 "Capacitor_SMD:C_0603_1608Metric" H 3938 4700 50  0001 C CNN
@@
 AR Path="/5FD1935C/5F64B0A6" Ref="Q4"  Part="1"
 AR Path="/5FD19389/5F64B0A6" Ref="Q7"  Part="1"
-F 0 "Q19" H 7900 1617 50  0000 C CNN
+F 0 "Q1" H 7900 1617 50  0000 C CNN
 F 1 "SISS23DN-T1-GE3" H 7900 1526 50  0000 C CNN
 F 2 "mypartsLib:POWERPAK-1212-8" H 7900 800 50  0001 C CNN
@@
 AR Path="/5FD1935C/5F671DB4" Ref="R38"  Part="1"
 AR Path="/5FD19389/5F671DB4" Ref="R49"  Part="1"
-F 0 "R86" H 7000 1750 50  0000 L CNN
+F 0 "R27" H 7000 1750 50  0000 L CNN
 F 1 "100k" H 7000 1550 50  0000 L CNN
 F 2 "Resistor_SMD:R_0603_1608Metric" V 6880 1650 50  0001 C CNN
@@
 AR Path="/5FD1935C/5F67CD1A" Ref="R41"  Part="1"
 AR Path="/5FD19389/5F67CD1A" Ref="R52"  Part="1"
-F 0 "R89" H 9300 2250 50  0000 L CNN
+F 0 "R30" H 9300 2250 50  0000 L CNN
 F 1 "100k" H 9300 2050 50  0000 L CNN
 F 2 "Resistor_SMD:R_0603_1608Metric" V 9180 2150 50  0001 C CNN
@@
 AR Path="/5FD1935C/5F6AFC79" Ref="R40"  Part="1"
 AR Path="/5FD19389/5F6AFC79" Ref="R51"  Part="1"
-F 0 "R88" H 8850 5000 50  0000 L CNN
+F 0 "R29" H 8850 5000 50  0000 L CNN
 F 1 "10k" H 8850 4800 50  0000 L CNN
 F 2 "Resistor_SMD:R_0603_1608Metric" V 8730 4900 50  0001 C CNN
@@
 AR Path="/5FD1935C/60873814" Ref="RV2"  Part="1"
 AR Path="/5FD19389/60873814" Ref="RV3"  Part="1"
-F 0 "RV6" H 3431 2846 50  0000 R CNN
+F 0 "RV1" H 3431 2846 50  0000 R CNN
 F 1 "200k" H 3431 2755 50  0000 R CNN
 F 2 "Potentiometer_SMD:Potentiometer_Bourns_3314G_Vertical" H 3500 2800 50  0001 C CNN
@@
 AR Path="/5FD1935C/5FD0BC61" Ref="Q6"  Part="1"
 AR Path="/5FD19389/5FD0BC61" Ref="Q9"  Part="1"
-F 0 "Q21" H 9294 4646 50  0000 L CNN
+F 0 "Q3" H 9294 4646 50  0000 L CNN
 F 1 "BC848B" H 9294 4555 50  0000 L CNN
 F 2 "Package_TO_SOT_SMD:SOT-23" H 8950 5100 50  0001 L CNN
@@
 AR Path="/5FD1935C/5FD2B5C8" Ref="CR6"  Part="1"
 AR Path="/5FD19389/5FD2B5C8" Ref="CR10"  Part="1"
-F 0 "CR24" V 6356 2046 50  0000 R CNN
+F 0 "CR2" V 6356 2046 50  0000 R CNN
 F 1 "1SS352_H3FT" V 6250 2046 50  0000 R CNN
 F 2 "mypartsLib:1SS352_H3FT" H 6250 1900 60  0001 C CNN
@@
 AR Path="/5FD1935C/5FD2B5C9" Ref="CR5"  Part="1"
 AR Path="/5FD19389/5FD2B5C9" Ref="CR9"  Part="1"
-F 0 "CR23" V 4356 3096 50  0000 R CNN
+F 0 "CR1" V 4356 3096 50  0000 R CNN
 F 1 "1SS352_H3FT" V 4250 3096 50  0000 R CNN
 F 2 "mypartsLib:1SS352_H3FT" H 4250 2950 60  0001 C CNN
@@
 AR Path="/5FD1935C/5FD0BC60" Ref="Q5"  Part="1"
 AR Path="/5FD19389/5FD0BC60" Ref="Q8"  Part="1"
-F 0 "Q20" H 7705 2404 50  0000 L CNN
+F 0 "Q2" H 7705 2404 50  0000 L CNN
 F 1 "IRF7404" H 7705 2495 50  0000 L CNN
 F 2 "Package_SO:SOIC-8_3.9x4.9mm_P1.27mm" H 7700 2375 50  0001 L CIN
@@
 AR Path="/5FD1935C/5FD0BC62" Ref="CR8"  Part="1"
 AR Path="/5FD19389/5FD0BC62" Ref="CR12"  Part="1"
-F 0 "CR26" H 7700 4700 50  0000 R CNN
+F 0 "CR4" H 7700 4700 50  0000 R CNN
 F 1 "1SS352_H3FT" H 7900 4800 50  0000 R CNN
 F 2 "mypartsLib:1SS352_H3FT" H 7650 4700 60  0001 C CNN
@@
 AR Path="/5FD1935C/5FD0BC63" Ref="CR7"  Part="1"
 AR Path="/5FD19389/5FD0BC63" Ref="CR11"  Part="1"
-F 0 "CR25" H 7700 4850 50  0000 R CNN
+F 0 "CR3" H 7700 4850 50  0000 R CNN
 F 1 "1SS352_H3FT" H 7900 4750 50  0000 R CNN
 F 2 "mypartsLib:1SS352_H3FT" H 7650 4350 60  0001 C CNN
@@
 AR Path="/5FD1935C/5FD2B5D1" Ref="R39"  Part="1"
 AR Path="/5FD19389/5FD2B5D1" Ref="R50"  Part="1"
-F 0 "R87" V 8600 4550 50  0000 L CNN
+F 0 "R28" V 8600 4550 50  0000 L CNN
 F 1 "10k" V 8400 4550 50  0000 L CNN
 F 2 "Resistor_SMD:R_0603_1608Metric" V 8430 4600 50  0001 C CNN
@@
 AR Path="/5FD19389/5FD1BC90" Ref="IC3"  Part="1"
 AR Path="/5FD193BD/5FD1BC90" Ref="IC4"  Part="1"
-F 0 "IC6" H 5150 4865 50  0000 C CNN
+F 0 "IC1" H 5150 4865 50  0000 C CNN
 F 1 "OP191GSZ_v2" H 5150 4774 50  0000 C CNN
 F 2 "Package_SO:SOIC-8_3.9x4.9mm_P1.27mm" H 5750 4650 50  0001 L CNN
@@
 AR Path="/5FD1935C/5FD3743B" Ref="R31"  Part="1"
 AR Path="/5FD19389/5FD3743B" Ref="R42"  Part="1"
-F 0 "R79" H 2350 3100 50  0000 L CNN
+F 0 "R20" H 2350 3100 50  0000 L CNN
 F 1 "6k" H 2350 2900 50  0000 L CNN
 F 2 "Resistor_SMD:R_0603_1608Metric" V 2230 3000 50  0001 C CNN
@@
 AR Path="/5FD1935C/5FD25536" Ref="R34"  Part="1"
 AR Path="/5FD19389/5FD25536" Ref="R45"  Part="1"
-F 0 "R82" H 3550 3250 50  0000 L CNN
+F 0 "R23" H 3550 3250 50  0000 L CNN
 F 1 "50k" H 3550 3050 50  0000 L CNN
 F 2 "Resistor_SMD:R_0603_1608Metric" V 3430 3150 50  0001 C CNN

Commit message: PCB reUpdate
Parts:
- added R123: 1k, Resistor_SMD:R_0603_1608Metric, symbol Device:R
- R79: value 6k -> 5k
Connections:
- net INPUT: now also R123.1; no longer R79.1
- new net: R123.2, R79.1
Other:
- moved on the sheet: R20
Changed lines of the file:
@@
 	4700 3900 3500 3900
 Wire Wire Line
-	2300 3150 2300 3700
+	2300 3300 2300 3700
 Connection ~ 2300 3700
 Wire Wire Line
@@
 	4850 4600 5300 4600
 Wire Wire Line
-	2300 1650 2300 2850
+	2300 1650 2300 2650
 $Comp
 L Device:R R?
 U 1 1 5FD3743B
-P 2300 3000
+P 2300 3150
 AR Path="/5FD192D6/5FD3743B" Ref="R?"  Part="1"
 AR Path="/5FD19308/5FD3743B" Ref="R79"  Part="1"
@@
 AR Path="/5FD1935C/5FD3743B" Ref="R31"  Part="1"
 AR Path="/5FD19389/5FD3743B" Ref="R42"  Part="1"
-F 0 "R20" H 2350 3100 50  0000 L CNN
-F 1 "6k" H 2350 2900 50  0000 L CNN
-F 2 "Resistor_SMD:R_0603_1608Metric" V 2230 3000 50  0001 C CNN
-F 3 "~" H 2300 3000 50  0001 C CNN
-	1    2300 3000
+F 0 "R20" H 2350 3250 50  0000 L CNN
+F 1 "5k" H 2350 3050 50  0000 L CNN
+F 2 "Resistor_SMD:R_0603_1608Metric" V 2230 3150 50  0001 C CNN
+F 3 "~" H 2300 3150 50  0001 C CNN
+	1    2300 3150
 	1    0    0    -1
 $EndComp
@@
 Text Label 4580 1350 0    50   ~ 0
 Power_Line
+$Comp
+L Device:R R?
+U 1 1 5FD786EE
+P 2300 2800
+AR Path="/5FD192D6/5FD786EE" Ref="R?"  Part="1"
+AR Path="/5FD19308/5FD786EE" Ref="R123"  Part="1"
+AR Path="/5FD193BD/5FD786EE" Ref="R121"  Part="1"
+AR Path="/5FD19328/5FD786EE" Ref="R118"  Part="1"
+AR Path="/5FD1935C/5FD786EE" Ref="R119"  Part="1"
+AR Path="/5FD19389/5FD786EE" Ref="R120"  Part="1"
+F 0 "R118" H 2350 2900 50  0000 L CNN
+F 1 "1k" H 2350 2700 50  0000 L CNN
+F 2 "Resistor_SMD:R_0603_1608Metric" V 2230 2800 50  0001 C CNN
+F 3 "~" H 2300 2800 50  0001 C CNN
+	1    2300 2800
+	1    0    0    -1
+$EndComp
+Wire Wire Line
+	2300 2950 2300 3000
 $EndSCHEMATC
