File: rsp02_module_LoadSW_OCP_5_0V.sch (KiCad schematic (older format))
At the start: 23 parts, among them IC1 OP291GSZ_v2, Q1 SISS23DN-T1-GE3, Q2 IRF7404, Q3 BC848B

Commit message: Update
Parts:
- removed CR3, CR4: 1SS352_H3FT, mypartsLib:1SS352_H3FT, symbol mypartsLib:1SS352_H3FT
- removed Q2: IRF7404, Package_SO:SOIC-8_3.9x4.9mm_P1.27mm, symbol Transistor_FET:IRF7404
- added CR23, CR24: 1SS352_H3FT, mypartsLib:1SS352_H3FT, symbol mypartsLib:1SS352_H3FT
- added Q17: IRF7404, Package_SO:SOIC-8_3.9x4.9mm_P1.27mm, symbol Transistor_FET:IRF7404
- renumbered C1 to C16, C2 to C17, C3 to C18, CR1 to CR21, CR2 to CR22, IC1 to IC6, Q1 to Q16, Q3 to Q18, R1 to R65, R2 to R66, R3 to R67, R4 to R68, R5 to R69, R6 to R70, R9 to R71, R7 to R72, R8 to R73, RV1 to RV11, RV2 to RV12, Rh1 to Rh6
Connections:
- net LSWE1: now also CR23.2 (anode)
- net LSWE2: now also CR24.2 (anode)
- net at CR22.1 (cathode), R69.1: now also Q17.5 (D), Q17.6 (D), Q17.7 (D), Q17.8 (D)
- net at Q16.4 (G), R70.2: now also Q17.1 (S), Q17.2 (S), Q17.3 (S)
- net at Q18.3 (collector), R73.2: now also Q17.4 (G)
- net at R71.2: now also CR23.1 (cathode), CR24.1 (cathode)

Commit message: Update Design
Parts:
- removed IC6: OP291GSZ_v2, Package_SO:SOIC-8_3.9x4.9mm_P1.27mm, symbol mypartsLib:OP291GSZ_v2
- removed RV11: 100k, Potentiometer_SMD:Potentiometer_Bourns_3314G_Vertical, symbol Device:R_Potentiometer_Trim
- added IC5: OP191GSZ_v2, SOIC127P600X175-8N, symbol mypartsLib:OP191GSZ_v2
- added R68: 5.3k, Resistor_SMD:R_0402_1005Metric, symbol Device:R
- added R71: 50k, Resistor_SMD:R_0402_1005Metric, symbol Device:R
- R70: renamed from R66; value 0.5 -> 0.10
- RV5: renamed from RV12; value 100k -> 200k
- renumbered C16 to C13, C17 to C14, C18 to C15, CR21 to CR19, CR22 to CR20, CR23 to CR21, CR24 to CR22, R65 to R69, R67 to R72, R68 to R73, R69 to R74, R70 to R75, R71 to R76, R72 to R77, R73 to R78, Rh6 to Rh5
Connections:
- net GND: now also IC5.4 (-V)
- net INPUT: now also IC5.7 (+V), R68.1
- net at R69.1, Rh5.2: now also IC5.3 (+INA), R68.2
- net at CR20.2 (anode), R73.2, Rh5.1: now also IC5.6 (OUTA)
- net at C13.1, CR19.2 (anode), R72.1: now also IC5.2 (-INA), R71.2; no longer RV5.3
- new net: R71.1, RV5.3
- no-connect marks 3 -> 0
Other:
- moved on the sheet: C14, RV5

Commit message: Update PCB
Parts:
- C13, C14, C15: footprint Capacitor_SMD:C_0402_1005Metric -> Capacitor_SMD:C_0603_1608Metric
- IC5: footprint SOIC127P600X175-8N -> Package_SO:SOIC-8_3.9x4.9mm_P1.27mm
- R68, R69, R71, R72, R73, R74, R75, R76, R77, R78, Rh5: footprint Resistor_SMD:R_0402_1005Metric -> Resistor_SMD:R_0603_1608Metric
Changed lines of the file:
@@
 F 0 "R72" H 3550 4950 50  0000 L CNN
 F 1 "1000k" H 3550 4750 50  0000 L CNN
-F 2 "Resistor_SMD:R_0402_1005Metric" V 3430 4850 50  0001 C CNN
+F 2 "Resistor_SMD:R_0603_1608Metric" V 3430 4850 50  0001 C CNN
 F 3 "~" H 3500 4850 50  0001 C CNN
 	1    3500 4850
@@
 F 0 "C14" H 4950 5350 50  0000 L CNN
 F 1 "0.1u" H 4950 5150 50  0000 L CNN
-F 2 "Capacitor_SMD:C_0402_1005Metric" H 4888 5100 50  0001 C CNN
+F 2 "Capacitor_SMD:C_0603_1608Metric" H 4888 5100 50  0001 C CNN
 F 3 "~" H 4850 5250 50  0001 C CNN
 	1    4850 5250
@@
 F 0 "R74" H 6700 3050 50  0000 L CNN
 F 1 "1k" H 6700 2850 50  0000 L CNN
-F 2 "Resistor_SMD:R_0402_1005Metric" V 6580 2950 50  0001 C CNN
+F 2 "Resistor_SMD:R_0603_1608Metric" V 6580 2950 50  0001 C CNN
 F 3 "~" H 6650 2950 50  0001 C CNN
 	1    6650 2950
@@
 F 0 "Rh5" V 4500 2100 50  0000 L CNN
 F 1 "100k" V 4700 2050 50  0000 L CNN
-F 2 "Resistor_SMD:R_0402_1005Metric" V 4530 2150 50  0001 C CNN
+F 2 "Resistor_SMD:R_0603_1608Metric" V 4530 2150 50  0001 C CNN
 F 3 "~" H 4600 2150 50  0001 C CNN
 	1    4600 2150
@@
 F 0 "C15" V 7500 3750 50  0000 L CNN
 F 1 "0.1u" V 7800 3750 50  0000 L CNN
-F 2 "Capacitor_SMD:C_0402_1005Metric" H 7688 3650 50  0001 C CNN
+F 2 "Capacitor_SMD:C_0603_1608Metric" H 7688 3650 50  0001 C CNN
 F 3 "~" H 7650 3800 50  0001 C CNN
 	1    7650 3800
@@
 F 0 "R73" V 6150 3750 50  0000 L CNN
 F 1 "10k" V 6350 3750 50  0000 L CNN
-F 2 "Resistor_SMD:R_0402_1005Metric" V 6180 3800 50  0001 C CNN
+F 2 "Resistor_SMD:R_0603_1608Metric" V 6180 3800 50  0001 C CNN
 F 3 "~" H 6250 3800 50  0001 C CNN
 	1    6250 3800
@@
 F 0 "R69" H 2350 4950 50  0000 L CNN
 F 1 "100k" H 2350 4750 50  0000 L CNN
-F 2 "Resistor_SMD:R_0402_1005Metric" V 2230 4850 50  0001 C CNN
+F 2 "Resistor_SMD:R_0603_1608Metric" V 2230 4850 50  0001 C CNN
 F 3 "~" H 2300 4850 50  0001 C CNN
 	1    2300 4850
@@
 F 0 "C13" H 4000 4950 50  0000 L CNN
 F 1 "0.1u" H 4000 4750 50  0000 L CNN
-F 2 "Capacitor_SMD:C_0402_1005Metric" H 3938 4700 50  0001 C CNN
+F 2 "Capacitor_SMD:C_0603_1608Metric" H 3938 4700 50  0001 C CNN
 F 3 "~" H 3900 4850 50  0001 C CNN
 	1    3900 4850
@@
 F 0 "R75" H 7000 1750 50  0000 L CNN
 F 1 "100k" H 7000 1550 50  0000 L CNN
-F 2 "Resistor_SMD:R_0402_1005Metric" V 6880 1650 50  0001 C CNN
+F 2 "Resistor_SMD:R_0603_1608Metric" V 6880 1650 50  0001 C CNN
 F 3 "~" H 6950 1650 50  0001 C CNN
 	1    6950 1650
@@
 F 0 "R78" H 9300 2250 50  0000 L CNN
 F 1 "100k" H 9300 2050 50  0000 L CNN
-F 2 "Resistor_SMD:R_0402_1005Metric" V 9180 2150 50  0001 C CNN
+F 2 "Resistor_SMD:R_0603_1608Metric" V 9180 2150 50  0001 C CNN
 F 3 "~" H 9250 2150 50  0001 C CNN
 	1    9250 2150
@@
 F 0 "R77" H 8850 5000 50  0000 L CNN
 F 1 "10k" H 8850 4800 50  0000 L CNN
-F 2 "Resistor_SMD:R_0402_1005Metric" V 8730 4900 50  0001 C CNN
+F 2 "Resistor_SMD:R_0603_1608Metric" V 8730 4900 50  0001 C CNN
 F 3 "~" H 8800 4900 50  0001 C CNN
 	1    8800 4900
@@
 F 0 "R76" V 8600 4550 50  0000 L CNN
 F 1 "10k" V 8400 4550 50  0000 L CNN
-F 2 "Resistor_SMD:R_0402_1005Metric" V 8430 4600 50  0001 C CNN
+F 2 "Resistor_SMD:R_0603_1608Metric" V 8430 4600 50  0001 C CNN
 F 3 "~" H 8500 4600 50  0001 C CNN
 	1    8500 4600
@@
 F 0 "R68" H 2350 3100 50  0000 L CNN
 F 1 "5.3k" H 2350 2900 50  0000 L CNN
-F 2 "Resistor_SMD:R_0402_1005Metric" V 2230 3000 50  0001 C CNN
+F 2 "Resistor_SMD:R_0603_1608Metric" V 2230 3000 50  0001 C CNN
 F 3 "~" H 2300 3000 50  0001 C CNN
 	1    2300 3000
@@
 F 0 "IC5" H 5150 4865 50  0000 C CNN
 F 1 "OP191GSZ_v2" H 5150 4774 50  0000 C CNN
-F 2 "SOIC127P600X175-8N" H 5750 4650 50  0001 L CNN
+F 2 "Package_SO:SOIC-8_3.9x4.9mm_P1.27mm" H 5750 4650 50  0001 L CNN
 F 3 "http://uk.rs-online.com/web/p/products/0427284P" H 5700 4350 50  0001 L CNN
 F 4 "Analog Devices OP191GSZ Op Amp, 3MHz Rail-Rail, 3  9 V, 8-Pin SOIC" H 5750 4450 50  0001 L CNN "Description"
@@
 F 0 "R71" H 3550 3250 50  0000 L CNN
 F 1 "50k" H 3550 3050 50  0000 L CNN
-F 2 "Resistor_SMD:R_0402_1005Metric" V 3430 3150 50  0001 C CNN
+F 2 "Resistor_SMD:R_0603_1608Metric" V 3430 3150 50  0001 C CNN
 F 3 "~" H 3500 3150 50  0001 C CNN
 	1    3500 3150

Commit message: PCB Update
Connections:
- net Power_Line: now reaches CR19.1 (cathode), Q16.1 (S(1)), Q16.2 (S(2)), Q16.3 (S(3)), R70.1, R75.1, RV5.1, RV5.2
Changed lines of the file:
@@
 Wire Wire Line
 	3500 3000 3500 2950
+Text Label 4590 1350 0    50   ~ 0
+Power_Line
 $EndSCHEMATC

Commit message: PCB reUpdate
Parts:
- added R122: 300, Resistor_SMD:R_0603_1608Metric, symbol Device:R
- R68: value 5.3k -> 5k
Connections:
- net INPUT: now also R122.1; no longer R68.1
- new net: R122.2, R68.1
Other:
- moved on the sheet: R68
Changed lines of the file:
@@
 	4700 3900 3500 3900
 Wire Wire Line
-	2300 3150 2300 3700
+	2300 3300 2300 3700
 Connection ~ 2300 3700
 Wire Wire Line
@@
 OUTPUT
 Wire Wire Line
-	2300 1650 2300 2850
+	2300 1650 2300 2660
 $Comp
 L Device:R R68
 U 1 1 60894A4E
-P 2300 3000
+P 2300 3150
 AR Path="/5FD192D6/60894A4E" Ref="R68"  Part="1"
 AR Path="/5FD19308/60894A4E" Ref="R?"  Part="1"
 AR Path="/5FD193BD/60894A4E" Ref="R?"  Part="1"
 AR Path="/5FD19328/60894A4E" Ref="R?"  Part="1"
-F 0 "R68" H 2350 3100 50  0000 L CNN
-F 1 "5.3k" H 2350 2900 50  0000 L CNN
-F 2 "Resistor_SMD:R_0603_1608Metric" V 2230 3000 50  0001 C CNN
-F 3 "~" H 2300 3000 50  0001 C CNN
-	1    2300 3000
+F 0 "R68" H 2350 3250 50  0000 L CNN
+F 1 "5k" H 2350 3050 50  0000 L CNN
+F 2 "Resistor_SMD:R_0603_1608Metric" V 2230 3150 50  0001 C CNN
+F 3 "~" H 2300 3150 50  0001 C CNN
+	1    2300 3150
 	1    0    0    -1
 $EndComp
@@
 Text Label 4590 1350 0    50   ~ 0
 Power_Line
+$Comp
+L Device:R R122
+U 1 1 5FD69D33
+P 2300 2810
+AR Path="/5FD192D6/5FD69D33" Ref="R122"  Part="1"
+AR Path="/5FD19308/5FD69D33" Ref="R?"  Part="1"
+AR Path="/5FD193BD/5FD69D33" Ref="R?"  Part="1"
+AR Path="/5FD19328/5FD69D33" Ref="R?"  Part="1"
+F 0 "R122" H 2350 2910 50  0000 L CNN
+F 1 "300" H 2350 2710 50  0000 L CNN
+F 2 "Resistor_SMD:R_0603_1608Metric" V 2230 2810 50  0001 C CNN
+F 3 "~" H 2300 2810 50  0001 C CNN
+	1    2300 2810
+	1    0    0    -1
+$EndComp
+Wire Wire Line
+	2300 2960 2300 3000
 $EndSCHEMATC
